File: pcbs/touch_keyboard/touch_kb1/touch_kb1.kicad_pcb (KiCad board)
At the start: 2 copper layers, 229 x 104.5 mm, 69 parts, among them J1 Conn_01x05_Female, U1 74HC165, U2 74HC165, U3 74HC165, U4 74HC165

Commit message: Updates
Routing:
- net +3V3: track 365.7 -> 375.9 mm, vias 6 -> 11
- net Net-(R15-Pad2): track 99.2 -> 102.1 mm
- net Net-(R17-Pad2): track 50.1 -> 51.3 mm
- net SERDAT_OUT_1: track 127.3 -> 128.3 mm
- net (no net): vias 0 -> 6
Other:
- board text added: "-"
- board text added: "."
- board text added: "0"
- board text added: "1"
- board text added: "2"
- board text added: "3"
- board text added: "3V3"
- board text added: "4"
- board text added: "5"
- board text added: "6"
- board text added: "7"
- board text added: "8"
- board text added: "9"
- board text added: "A"
- board text added: "B"
- board text added: "C"
- board text added: "CLEAR"
- board text added: "CLK"
- board text added: "DECR ADDR"
- board text added: "DUMP"
- board text added: "Experimental School's Computer May 2024 menadue@gmail.com V1.0"
- board text added: "GND"
- board text added: "KI RESET"
- board text added: "LOAD"
- board text added: "NORM RESET"
- board text added: "RELOAD"
- board text added: "RUN"
- board text added: "SERDAT"
- board text added: "STOP"
