File: pcbs/touch_keyboard/touch_with_qt/overlay1/overlay1.kicad_pcb (KiCad board)
At the start: 2 copper layers, 229 x 104.5 mm, 0 parts

Commit message: Updates
Other:
- board text added: "CHECK"
- board text added: "Experimental School's Computer May 2024 menadue@gmail.com V1.0"
- board text removed: "Experimental School's Computer Keyboard Overlay May 2024 menadue@gmail.com V1.0"
Changed lines of the file:
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@@
   (page A4)
   (layers
-    (0 F.Cu signal hide)
+    (0 F.Cu signal)
     (31 B.Cu signal)
     (32 B.Adhes user)
-    (33 F.Adhes user hide)
+    (33 F.Adhes user)
     (34 B.Paste user)
     (35 F.Paste user)
@@
     (45 Margin user)
     (46 B.CrtYd user)
-    (47 F.CrtYd user)
+    (47 F.CrtYd user hide)
     (48 B.Fab user)
-    (49 F.Fab user)
+    (49 F.Fab user hide)
   )
   (setup
@@
     (via_min_size 0.4)
     (via_min_drill 0.3)
+    (user_via 0.6 0.4)
     (user_via 3.5 3.1)
     (uvia_size 0.3)
@@
       (drillshape 0)
       (scaleselection 1)
-      (outputdirectory "/tree/projects/github/experimental-computer-for-schools/pcbs/touch_keyboard/touch_with_qt/overlay1/fab1/"))
+      (outputdirectory "fab1/"))
   )
   (net 0 "")
@@
     (uvia_drill 0.1)
   )
-  (gr_text "LOAD\nSTORE" (at 66.3904 77.3312) (layer F.SilkS)
+  (gr_text RELOAD (at 216.5 107.875) (layer F.SilkS)
     (effects (font (size 2 2) (thickness 0.3)))
   )
-  (gr_text "Experimental School's Computer\nKeyboard Overlay\nMay 2024\nmenadue@gmail.com\nV1.0" (at 226.8 122.4) (layer B.SilkS)
-    (effects (font (size 1 1) (thickness 0.15)) (justify mirror))
-  )
-  (gr_text RELOAD (at 216.352 107.7604) (layer F.SilkS)
-    (effects (font (size 2 2) (thickness 0.3)))
-  )
-  (gr_text DUMP (at 226.1564 92.876) (layer F.SilkS)
-    (effects (font (size 2 2) (thickness 0.3)))
-  )
-  (gr_text DUMP (at 216.5044 77.89) (layer F.SilkS)
+  (gr_text "KI\nRESET" (at 171.394 107.4556) (layer F.SilkS)
     (effects (font (size 2 2) (thickness 0.3)))
   )
   (gr_text C (at 178.7092 92.7744) (layer F.SilkS)
     (effects (font (size 4 4) (thickness 0.6)))
+  )
+  (gr_text STOP (at 186.4816 77.8392) (layer F.SilkS)
+    (effects (font (size 2 2) (thickness 0.3)))
   )
   (gr_text B (at 171.394 77.7884) (layer F.SilkS)
@@
     (effects (font (size 4 4) (thickness 0.6)))
   )
-  (gr_text "KI\nRESET" (at 171.394 107.4556) (layer F.SilkS)
+  (gr_text RUN (at 178.7092 62.7516) (layer F.SilkS)
     (effects (font (size 2 2) (thickness 0.3)))
   )
-  (gr_text STOP (at 186.4816 77.8392) (layer F.SilkS)
+  (gr_text DUMP (at 216.5044 77.89) (layer F.SilkS)
     (effects (font (size 2 2) (thickness 0.3)))
   )
-  (gr_text RUN (at 178.7092 62.7516) (layer F.SilkS)
+  (gr_text CHECK (at 206.9 93.05) (layer F.SilkS)
     (effects (font (size 2 2) (thickness 0.3)))
+  )
+  (gr_text 4 (at 103.4236 92.9776) (layer F.SilkS)
+    (effects (font (size 4 4) (thickness 0.6)))
+  )
+  (gr_text 5 (at 118.9684 92.8252) (layer F.SilkS)
+    (effects (font (size 4 4) (thickness 0.6)))
+  )
+  (gr_text 6 (at 133.9544 92.9776) (layer F.SilkS)
+    (effects (font (size 4 4) (thickness 0.6)))
   )
   (gr_text 0 (at 141.422 107.7604) (layer F.SilkS)
@@
     (effects (font (size 4 4) (thickness 0.6)))
   )
-  (gr_text 6 (at 133.9544 92.9776) (layer F.SilkS)
+  (gr_text 1 (at 96.3116 77.4836) (layer F.SilkS)
     (effects (font (size 4 4) (thickness 0.6)))
   )
-  (gr_text 5 (at 118.9684 92.8252) (layer F.SilkS)
-    (effects (font (size 4 4) (thickness 0.6)))
-  )
-  (gr_text 4 (at 103.4236 92.9776) (layer F.SilkS)
+  (gr_text 2 (at 111.196 77.3312) (layer F.SilkS)
     (effects (font (size 4 4) (thickness 0.6)))
   )
@@
     (effects (font (size 4 4) (thickness 0.6)))
   )
-  (gr_text 2 (at 111.196 77.3312) (layer F.SilkS)
-    (effects (font (size 4 4) (thickness 0.6)))
-  )
-  (gr_text 1 (at 96.3116 77.4836) (layer F.SilkS)
-    (effects (font (size 4 4) (thickness 0.6)))
-  )
-  (gr_text . (at 133.9544 60.364) (layer F.SilkS)
-    (effects (font (size 6 6) (thickness 1)))
-  )
-  (gr_text - (at 118.7652 62.5484) (layer F.SilkS)
-    (effects (font (size 4 4) (thickness 0.6)))
-  )
-  (gr_text CLEAR (at 103.7792 62.8532) (layer F.SilkS)
-    (effects (font (size 2 2) (thickness 0.3)))
-  )
-  (gr_text "NORM\nRESET" (at 66.3396 107.2016) (layer F.SilkS)
-    (effects (font (size 2 2) (thickness 0.3)))
-  )
   (gr_text "INCR\nADDR" (at 73.7564 92.4188) (layer F.SilkS)
     (effects (font (size 2 2) (thickness 0.3)))
   )
   (gr_text "DECR\nADDR" (at 58.8212 92.7744) (layer F.SilkS)
+    (effects (font (size 2 2) (thickness 0.3)))
+  )
+  (gr_text "LOAD\nSTORE" (at 66.3904 77.3312) (layer F.SilkS)
+    (effects (font (size 2 2) (thickness 0.3)))
+  )
+  (gr_text "NORM\nRESET" (at 66.3396 107.2016) (layer F.SilkS)
     (effects (font (size 2 2) (thickness 0.3)))
   )
@@
     (effects (font (size 2 2) (thickness 0.3)))
   )
+  (gr_text CLEAR (at 103.7792 62.8532) (layer F.SilkS)
+    (effects (font (size 2 2) (thickness 0.3)))
+  )
+  (gr_text - (at 118.7652 62.5484) (layer F.SilkS)
+    (effects (font (size 4 4) (thickness 0.6)))
+  )
+  (gr_text . (at 133.9544 60.364) (layer F.SilkS)
+    (effects (font (size 6 6) (thickness 1)))
+  )
+  (gr_text "Experimental School's Computer\nMay 2024\nmenadue@gmail.com\nV1.0" (at 306.2 70.4) (layer B.SilkS)
+    (effects (font (size 1 1) (thickness 0.15)) (justify mirror))
+  )
   (gr_line (start 28.9 145.2) (end 29.9 145.2) (layer Edge.Cuts) (width 0.05))
