File: pcbs/desktop_esc/desktop_esc/information.sch (KiCad schematic (older format))
At the start: 0 parts

Commit message: Updates
Other:
- note added: "Desktop ESC has the same hardware layout as the small ESC,\nexcept there's no local keyboard. Instead there's a connection to \nthe AT42QT1418 touch PCB. The OLED display is not present, as a \nlarger LCD is used for the TV replica. The keboard scanning GPIOs \nare used to drive the LCD and the touch keyboard interfaces.\n"
- note added: "Desktop replica has no OLED display so it can be used \nusing USB to generate keypresses and see the display.\n"
- note removed: "Desktop ESC has the same hardware layout as the small ESC,\nexcept there's no local keyboard. Instead there's a connection to \nthe AT42QT1418 touch PCB. The OLED display is driven, as is a \nlarger LCD for the TV replica. The keboard scanning GPIOs are used\nto drive the LCD and the touch keyboard interfaces.\n"
Changed lines of the file:
@@
 $Descr A4 11693 8268
 encoding utf-8
-Sheet 2 2
+Sheet 2 3
 Title ""
 Date ""
@@
 Power Budget\n\nLCD Module Logic:  80mA\nLD backlight        :   200mA\nOLED                   :\nPico                     :\nSD card               :\nTouch Keyboard  :\n
 Text Notes 3225 1175 0    50   ~ 0
-Desktop ESC has the same hardware layout as the small ESC,\nexcept there's no local keyboard. Instead there's a connection to \nthe AT42QT1418 touch PCB. The OLED display is driven, as is a \nlarger LCD for the TV replica. The keboard scanning GPIOs are used\nto drive the LCD and the touch keyboard interfaces.\n
+Desktop ESC has the same hardware layout as the small ESC,\nexcept there's no local keyboard. Instead there's a connection to \nthe AT42QT1418 touch PCB. The OLED display is not present, as a \nlarger LCD is used for the TV replica. The keboard scanning GPIOs \nare used to drive the LCD and the touch keyboard interfaces.\n
+Text Notes 3200 1600 0    50   ~ 0
+Desktop replica has no OLED display so it can be used \nusing USB to generate keypresses and see the  display.\n
 $EndSCHEMATC
