File: pcbs/desktop_esc/desktop_esc/level_shift.sch (KiCad schematic (older format))
At the start: 4 parts, among them U3 ajm_cd40109, U4 ajm_cd40109, U5 ajm_cd40109, U6 ajm_cd40109

Commit message: Updates
Parts:
- added C10, C11, C12, C13, C14, C8, C9: 100nF, Capacitor_SMD:C_0805_2012Metric_Pad1.18x1.45mm_HandSolder, symbol Device:C
- added C7: 100nGF, Capacitor_SMD:C_0805_2012Metric_Pad1.18x1.45mm_HandSolder, symbol Device:C
- added JP7: 40109_B_GND, Jumper:SolderJumper-2_P1.3mm_Bridged_RoundedPad1.0x1.5mm, symbol Device:Jumper_NO_Small
- added JP8: 40109_C_GND, Jumper:SolderJumper-2_P1.3mm_Bridged_RoundedPad1.0x1.5mm, symbol Device:Jumper_NO_Small
- added JP9: 40109_D_GND, Jumper:SolderJumper-2_P1.3mm_Bridged_RoundedPad1.0x1.5mm, symbol Device:Jumper_NO_Small
- U3, U4, U5, U6: footprint (none) -> Package_SO:SOP-24_7.5x15.4mm_P1.27mm
Connections:
- net +3V3: now also C11.1, C13.1, C7.1, C9.1
- net +5V: now also C10.1, C12.1, C14.1, C8.1
- net GND: now also C10.2, C11.2, C12.2, C13.2, C14.2, C7.2, C8.2, C9.2, JP7.2, JP8.2, JP9.2
- net at U6.6: now also JP7.1
- net at U6.10: now also JP8.1
- net at U6.14: now also JP9.1

Commit message: Updates
Parts:
- U3, U4, U5, U6: footprint Package_SO:SOP-24_7.5x15.4mm_P1.27mm -> Package_SO:SOIC-16W_7.5x10.3mm_P1.27mm
Changed lines of the file:
@@
 F 0 "U3" H 1850 1225 50  0000 C CNN
 F 1 "ajm_cd40109" H 2000 1150 50  0000 C CNN
-F 2 "Package_SO:SOP-24_7.5x15.4mm_P1.27mm" H 1425 1250 50  0001 C CNN
+F 2 "Package_SO:SOIC-16W_7.5x10.3mm_P1.27mm" H 1425 1250 50  0001 C CNN
 F 3 "" H 1425 1250 50  0001 C CNN
 	1    1625 950
@@
 F 0 "U3" H 1825 1875 50  0000 C CNN
 F 1 "ajm_cd40109" H 1975 1775 50  0000 C CNN
-F 2 "Package_SO:SOP-24_7.5x15.4mm_P1.27mm" H 1425 1925 50  0001 C CNN
+F 2 "Package_SO:SOIC-16W_7.5x10.3mm_P1.27mm" H 1425 1925 50  0001 C CNN
 F 3 "" H 1425 1925 50  0001 C CNN
 	2    1625 1625
@@
 F 0 "U3" H 1875 2550 50  0000 C CNN
 F 1 "ajm_cd40109" H 1975 2475 50  0000 C CNN
-F 2 "Package_SO:SOP-24_7.5x15.4mm_P1.27mm" H 1425 2575 50  0001 C CNN
+F 2 "Package_SO:SOIC-16W_7.5x10.3mm_P1.27mm" H 1425 2575 50  0001 C CNN
 F 3 "" H 1425 2575 50  0001 C CNN
 	3    1625 2275
@@
 F 0 "U3" H 1950 3225 50  0000 C CNN
 F 1 "ajm_cd40109" H 2050 3125 50  0000 C CNN
-F 2 "Package_SO:SOP-24_7.5x15.4mm_P1.27mm" H 1450 3250 50  0001 C CNN
+F 2 "Package_SO:SOIC-16W_7.5x10.3mm_P1.27mm" H 1450 3250 50  0001 C CNN
 F 3 "" H 1450 3250 50  0001 C CNN
 	4    1650 2950
@@
 F 0 "U3" H 1850 2875 50  0000 R CNN
 F 1 "ajm_cd40109" H 1875 2800 50  0000 R CNN
-F 2 "Package_SO:SOP-24_7.5x15.4mm_P1.27mm" H 1475 4250 50  0001 C CNN
+F 2 "Package_SO:SOIC-16W_7.5x10.3mm_P1.27mm" H 1475 4250 50  0001 C CNN
 F 3 "" H 1475 4250 50  0001 C CNN
 	5    1675 3950
@@
 F 0 "U4" H 3400 1200 50  0000 C CNN
 F 1 "ajm_cd40109" H 3500 1125 50  0000 C CNN
-F 2 "Package_SO:SOP-24_7.5x15.4mm_P1.27mm" H 2975 1250 50  0001 C CNN
+F 2 "Package_SO:SOIC-16W_7.5x10.3mm_P1.27mm" H 2975 1250 50  0001 C CNN
 F 3 "" H 2975 1250 50  0001 C CNN
 	1    3175 950
@@
 F 0 "U4" H 3450 1875 50  0000 C CNN
 F 1 "ajm_cd40109" H 3600 1775 50  0000 C CNN
-F 2 "Package_SO:SOP-24_7.5x15.4mm_P1.27mm" H 2975 1925 50  0001 C CNN
+F 2 "Package_SO:SOIC-16W_7.5x10.3mm_P1.27mm" H 2975 1925 50  0001 C CNN
 F 3 "" H 2975 1925 50  0001 C CNN
 	2    3175 1625
@@
 F 0 "U4" H 3450 2575 50  0000 C CNN
 F 1 "ajm_cd40109" H 3550 2475 50  0000 C CNN
-F 2 "Package_SO:SOP-24_7.5x15.4mm_P1.27mm" H 2975 2575 50  0001 C CNN
+F 2 "Package_SO:SOIC-16W_7.5x10.3mm_P1.27mm" H 2975 2575 50  0001 C CNN
 F 3 "" H 2975 2575 50  0001 C CNN
 	3    3175 2275
@@
 F 0 "U4" H 3475 3225 50  0000 C CNN
 F 1 "ajm_cd40109" H 3600 3150 50  0000 C CNN
-F 2 "Package_SO:SOP-24_7.5x15.4mm_P1.27mm" H 3000 3250 50  0001 C CNN
+F 2 "Package_SO:SOIC-16W_7.5x10.3mm_P1.27mm" H 3000 3250 50  0001 C CNN
 F 3 "" H 3000 3250 50  0001 C CNN
 	4    3200 2950
@@
 F 0 "U5" H 5175 1275 50  0000 C CNN
 F 1 "ajm_cd40109" H 5275 1200 50  0000 C CNN
-F 2 "Package_SO:SOP-24_7.5x15.4mm_P1.27mm" H 4750 1275 50  0001 C CNN
+F 2 "Package_SO:SOIC-16W_7.5x10.3mm_P1.27mm" H 4750 1275 50  0001 C CNN
 F 3 "" H 4750 1275 50  0001 C CNN
 	1    4950 975
@@
 F 0 "U5" H 5200 1975 50  0000 C CNN
 F 1 "ajm_cd40109" H 5325 1900 50  0000 C CNN
-F 2 "Package_SO:SOP-24_7.5x15.4mm_P1.27mm" H 4750 1950 50  0001 C CNN
+F 2 "Package_SO:SOIC-16W_7.5x10.3mm_P1.27mm" H 4750 1950 50  0001 C CNN
 F 3 "" H 4750 1950 50  0001 C CNN
 	2    4950 1650
@@
 F 0 "U5" H 5150 2600 50  0000 C CNN
 F 1 "ajm_cd40109" H 5300 2525 50  0000 C CNN
-F 2 "Package_SO:SOP-24_7.5x15.4mm_P1.27mm" H 4750 2600 50  0001 C CNN
+F 2 "Package_SO:SOIC-16W_7.5x10.3mm_P1.27mm" H 4750 2600 50  0001 C CNN
 F 3 "" H 4750 2600 50  0001 C CNN
 	3    4950 2300
@@
 F 0 "U5" H 5175 3275 50  0000 C CNN
 F 1 "ajm_cd40109" H 5300 3200 50  0000 C CNN
-F 2 "Package_SO:SOP-24_7.5x15.4mm_P1.27mm" H 4775 3275 50  0001 C CNN
+F 2 "Package_SO:SOIC-16W_7.5x10.3mm_P1.27mm" H 4775 3275 50  0001 C CNN
 F 3 "" H 4775 3275 50  0001 C CNN
 	4    4975 2975
@@
 F 0 "U6" H 7075 1300 50  0000 C CNN
 F 1 "ajm_cd40109" H 7225 1225 50  0000 C CNN
-F 2 "Package_SO:SOP-24_7.5x15.4mm_P1.27mm" H 6700 1300 50  0001 C CNN
+F 2 "Package_SO:SOIC-16W_7.5x10.3mm_P1.27mm" H 6700 1300 50  0001 C CNN
 F 3 "" H 6700 1300 50  0001 C CNN
 	1    6900 1000
@@
 F 0 "U6" H 7100 1975 50  0000 C CNN
 F 1 "ajm_cd40109" H 7250 1900 50  0000 C CNN
-F 2 "Package_SO:SOP-24_7.5x15.4mm_P1.27mm" H 6700 1975 50  0001 C CNN
+F 2 "Package_SO:SOIC-16W_7.5x10.3mm_P1.27mm" H 6700 1975 50  0001 C CNN
 F 3 "" H 6700 1975 50  0001 C CNN
 	2    6900 1675
@@
 F 0 "U6" H 7100 2625 50  0000 C CNN
 F 1 "ajm_cd40109" H 7250 2550 50  0000 C CNN
-F 2 "Package_SO:SOP-24_7.5x15.4mm_P1.27mm" H 6700 2625 50  0001 C CNN
+F 2 "Package_SO:SOIC-16W_7.5x10.3mm_P1.27mm" H 6700 2625 50  0001 C CNN
 F 3 "" H 6700 2625 50  0001 C CNN
 	3    6900 2325
@@
 F 0 "U6" H 7125 3300 50  0000 C CNN
 F 1 "ajm_cd40109" H 7250 3225 50  0000 C CNN
-F 2 "Package_SO:SOP-24_7.5x15.4mm_P1.27mm" H 6725 3300 50  0001 C CNN
+F 2 "Package_SO:SOIC-16W_7.5x10.3mm_P1.27mm" H 6725 3300 50  0001 C CNN
 F 3 "" H 6725 3300 50  0001 C CNN
 	4    6925 3000
@@
 F 0 "U4" H 3100 3100 50  0000 R CNN
 F 1 "ajm_cd40109" H 3100 3000 50  0000 R CNN
-F 2 "Package_SO:SOP-24_7.5x15.4mm_P1.27mm" H 3125 4325 50  0001 C CNN
+F 2 "Package_SO:SOIC-16W_7.5x10.3mm_P1.27mm" H 3125 4325 50  0001 C CNN
 F 3 "" H 3125 4325 50  0001 C CNN
 	5    3325 4025
@@
 F 0 "U5" H 4900 3175 50  0000 R CNN
 F 1 "ajm_cd40109" H 4875 3075 50  0000 R CNN
-F 2 "Package_SO:SOP-24_7.5x15.4mm_P1.27mm" H 4850 4325 50  0001 C CNN
+F 2 "Package_SO:SOIC-16W_7.5x10.3mm_P1.27mm" H 4850 4325 50  0001 C CNN
 F 3 "" H 4850 4325 50  0001 C CNN
 	5    5050 4025
@@
 F 0 "U6" H 6825 3375 50  0000 R CNN
 F 1 "ajm_cd40109" H 6850 3225 50  0000 R CNN
-F 2 "Package_SO:SOP-24_7.5x15.4mm_P1.27mm" H 6800 4350 50  0001 C CNN
+F 2 "Package_SO:SOIC-16W_7.5x10.3mm_P1.27mm" H 6800 4350 50  0001 C CNN
 F 3 "" H 6800 4350 50  0001 C CNN
 	5    7000 4050

Commit message: Updates
Changed lines of the file:
@@
 	6900 4625 6900 4475
-$Comp
-L power:+5V #PWR0107
-U 1 1 6671749A
-P -500 1550
-F 0 "#PWR0107" H -500 1400 50  0001 C CNN
-F 1 "+5V" H -485 1723 50  0000 C CNN
-F 2 "" H -500 1550 50  0001 C CNN
-F 3 "" H -500 1550 50  0001 C CNN
-	1    -500 1550
-	1    0    0    -1
-$EndComp
 $Comp
 L power:+5V #PWR0109
