File: pcbs/desktop_esc/desktop_esc/desktop_esc.kicad_pcb (KiCad board)
At the start: 2 copper layers, 8 parts, among them J7 Conn_01x02_Female, U1 Pico, U2 AP1117-33

Commit message: Updates
Parts:
- added C10: 100nF, Capacitor_SMD:C_0805_2012Metric_Pad1.18x1.45mm_HandSolder, F.Cu at (34.9, 50.3)
- added C11: 100nF, Capacitor_SMD:C_0805_2012Metric_Pad1.18x1.45mm_HandSolder, F.Cu at (30.1, 47.3)
- added C12: 100nF, Capacitor_SMD:C_0805_2012Metric_Pad1.18x1.45mm_HandSolder, F.Cu at (44.5, 47.3)
- added C13: 100nF, Capacitor_SMD:C_0805_2012Metric_Pad1.18x1.45mm_HandSolder, F.Cu at (30.1, 56.3)
- added C14: 100nF, Capacitor_SMD:C_0805_2012Metric_Pad1.18x1.45mm_HandSolder, F.Cu at (30.1, 53.3)
- added C3: C_Small, Capacitor_SMD:C_0805_2012Metric_Pad1.18x1.45mm_HandSolder, F.Cu at (85.4, 39.9)
- added C4: C_Small, Capacitor_SMD:C_0805_2012Metric_Pad1.18x1.45mm_HandSolder, F.Cu at (80.6, 39.9)
- added C5: C_Small, Capacitor_SMD:C_0805_2012Metric_Pad1.18x1.45mm_HandSolder, F.Cu at (95.1, 39.9)
- added C6: C_Small, Capacitor_SMD:C_0805_2012Metric_Pad1.18x1.45mm_HandSolder, F.Cu at (90.3, 39.9)
- added C7: 100nGF, Capacitor_SMD:C_0805_2012Metric_Pad1.18x1.45mm_HandSolder, F.Cu at (34.9, 47.3)
- added C8: 100nF, Capacitor_SMD:C_0805_2012Metric_Pad1.18x1.45mm_HandSolder, F.Cu at (30.1, 50.3)
- added C9: 100nF, Capacitor_SMD:C_0805_2012Metric_Pad1.18x1.45mm_HandSolder, F.Cu at (39.7, 47.3)
- added J1: Conn_02x10_Odd_Even, Connector_IDC:IDC-Header_2x10_P2.54mm_Latch_Vertical, F.Cu at (130.9, 71.2)
- added J2: Conn_01x12_Female, Connector_PinHeader_2.54mm:PinHeader_1x12_P2.54mm_Vertical, F.Cu at (102.3, 100.9)
- added J3: Conn_01x03_Female, Connector_PinHeader_2.54mm:PinHeader_1x03_P2.54mm_Vertical, F.Cu at (124.1, 115.0)
- added JP1: TOUCH_CS, Jumper:SolderJumper-2_P1.3mm_Open_TrianglePad1.0x1.5mm, F.Cu at (93.5, 43.2)
- added JP2: TOUCH_RX, Jumper:SolderJumper-2_P1.3mm_Open_TrianglePad1.0x1.5mm, F.Cu at (89.1, 43.2)
- added JP3: TOUCH_MISO, Jumper:SolderJumper-2_P1.3mm_Open_TrianglePad1.0x1.5mm, F.Cu at (84.8, 43.2)
- added JP4: TOUCH_TX, Jumper:SolderJumper-2_P1.3mm_Open_TrianglePad1.0x1.5mm, F.Cu at (80.4, 43.2)
- added JP7: 40109_B_GND, Jumper:SolderJumper-2_P1.3mm_Bridged_RoundedPad1.0x1.5mm, F.Cu at (43.8, 50.6)
- added JP8: 40109_C_GND, Jumper:SolderJumper-2_P1.3mm_Bridged_RoundedPad1.0x1.5mm, F.Cu at (39.5, 50.6)
- added JP9: 40109_D_GND, Jumper:SolderJumper-2_P1.3mm_Bridged_RoundedPad1.0x1.5mm, F.Cu at (34.7, 53.6)
- added RV1: R_POT, Potentiometer_THT:Potentiometer_Bourns_3296W_Vertical, F.Cu at (110.9, 71.1)
- added U3: ajm_cd40109, Package_SO:SOP-24_7.5x15.4mm_P1.27mm, F.Cu at (153.6, 87.5)
- added U4: ajm_cd40109, Package_SO:SOP-24_7.5x15.4mm_P1.27mm, F.Cu at (132.6, 86.8)
- added U5: ajm_cd40109, Package_SO:SOP-24_7.5x15.4mm_P1.27mm, F.Cu at (175.1, 88.3)
- added U6: ajm_cd40109, Package_SO:SOP-24_7.5x15.4mm_P1.27mm, F.Cu at (110.4, 86.2)
- added XS1: 502p_SD_ebay-uSD-push_push_SMD, ajm_kicad:Conn_uSDcard, F.Cu at (178.5, 66.1)
- moved J7 94.5 mm to (117.8, 129.3), turned to 90 degrees
- moved D5 93.6 mm to (128.3, 133.2)
- moved JP5 93.6 mm to (133.4, 136.2)
- moved C1 93.6 mm to (133.6, 133.0)
- moved C2 93.6 mm to (138.3, 133.0)
- moved JP6 93.6 mm to (137.7, 136.2)
- moved U2 82.1 mm to (114.3, 115.5)
- moved U1 21.0 mm to (160.3, 112.8), turned to 270 degrees
Other:
- board outline added: 100 x 75 mm

Commit message: Updates
Parts:
- removed C3, C4, C5, C6: C_Small, Capacitor_SMD:C_0805_2012Metric_Pad1.18x1.45mm_HandSolder
- added JP10: Jumper_NC_Small, Jumper:SolderJumper-2_P1.3mm_Bridged_RoundedPad1.0x1.5mm, F.Cu at (191.1, 114.6)
- C10, C11, C12, C13, C14, C7, C8, C9: moved to B.Cu
- U3, U4, U5, U6: footprint Package_SO:SOP-24_7.5x15.4mm_P1.27mm -> Package_SO:SOIC-16W_7.5x10.3mm_P1.27mm
- moved C13 140.0 mm to (167.2, 84.9), turned to 90 degrees
- moved C14 137.6 mm to (164.1, 84.9), turned to 90 degrees
- moved JP8 135.8 mm to (168.3, 93.4), turned to 180 degrees
- moved JP9 133.4 mm to (166.1, 76.5), turned to 180 degrees
- moved JP7 127.9 mm to (164.3, 93.5)
- moved C10 116.7 mm to (146.3, 85.1), turned to 90 degrees
- moved C9 116.2 mm to (149.5, 85.2), turned to 90 degrees
- moved C8 103.8 mm to (127.9, 84.9), turned to 90 degrees
- moved C7 103.4 mm to (131.2, 85.0), turned to 90 degrees
- moved C11 92.1 mm to (114.1, 84.9), turned to 90 degrees
- moved JP3 76.9 mm to (105.7, 117.2)
- moved C12 76.3 mm to (110.8, 85.0), turned to 90 degrees
- moved JP4 68.8 mm to (105.6, 107.2)
- moved U5 65.2 mm to (110.0, 85.0)
- moved JP2 63.2 mm to (105.7, 104.2)
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Connections:
- J2 pad 11: (no net) -> DBG_CLK_3V3
- J2 pad 12: (no net) -> WS_3V3
- U1 pad 20: DBG_CLK_3V4 -> DBG_CLK_3V3
- U1 pad 22: WS_3V5 -> WS_3V3
Routing:
- net +5V: track 0.00 -> 261.2 mm, vias 0 -> 21
- net GND: track 0.00 -> 240.0 mm, vias 0 -> 17
- net +3V3: track 0.00 -> 187.2 mm, vias 0 -> 8
- net MISO_D0: track 0.00 -> 111.8 mm, vias 0 -> 2
- net SD_CLK: track 0.00 -> 111.0 mm, vias 0 -> 4
- net MOSI_DI: track 0.00 -> 110.8 mm, vias 0 -> 4
- net A0_3V3: track 0.00 -> 107.2 mm, vias 0 -> 6
- net SD_DAT1: track 0.00 -> 102.1 mm, vias 0 -> 4
- net RESET_N_3V3: track 0.00 -> 101.1 mm, vias 0 -> 2
- net VSYS: track 0.00 -> 97.3 mm, vias 0 -> 4
- net SCK_3V3: track 0.00 -> 77.5 mm, vias 0 -> 5
- net SD_DAT2: track 0.00 -> 75.7 mm, vias 0 -> 2
- net DB2_3V3: track 0.00 -> 74.6 mm, vias 0 -> 4
- net DB0_3V3: track 0.00 -> 73.3 mm, vias 0 -> 2
- net DB3_3V3: track 0.00 -> 73.2 mm, vias 0 -> 4
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- added copper zone on B.Cu, net GND
Other:
- board text added: "Experimental School's Computer Desktop Touch Keyboard V1.0 May 2024 menadue@gmail.com"

Commit message: Updates
Parts:
- added C3: 150pF, Capacitor_SMD:C_0805_2012Metric_Pad1.18x1.45mm_HandSolder, F.Cu at (175.5, 71.6)
- added C4: 150pF, Capacitor_SMD:C_0805_2012Metric_Pad1.18x1.45mm_HandSolder, F.Cu at (157.4, 71.6)
- added C5: 150pF, Capacitor_SMD:C_0805_2012Metric_Pad1.18x1.45mm_HandSolder, F.Cu at (171.3, 71.5)
- added C6: 150pF, Capacitor_SMD:C_0805_2012Metric_Pad1.18x1.45mm_HandSolder, F.Cu at (161.9, 71.7)
- RV1: value R_POT -> 20k
- moved J1 45.9 mm to (176.5, 62.5), turned to 270 degrees
- moved XS1 18.3 mm to (190.7, 78.2), turned to 90 degrees
Connections:
- J2 pad 7: MOSI_3V3 -> (no net)
- J2 pad 9: MISO_3V3 -> (no net)
- JP1 pad 1: (no net) -> CS_N_3V3
- JP3 pad 1: MISO_3V3 -> (no net)
- U1 pad 15: MOSI_3V3 -> A0_3V3
- U1 pad 35: A0_3V3 -> Net-(U1-Pad35)
Routing:
- net CS_N_3V3: track 32.9 -> 97.8 mm, vias 0 -> 2
- net MOSI_3V3: track 60.3 -> 0.00 mm, vias 1 -> 0
- net Net-(J1-Pad3): track 28.0 -> 73.0 mm
- net RD_N_5V: track 52.5 -> 96.6 mm, vias 1 -> 3
- net A0_3V3: track 107.2 -> 63.8 mm, vias 6 -> 3
- net WR_N_5V: track 49.4 -> 88.1 mm, vias 1 -> 4
- net DB0_5V: track 34.7 -> 69.2 mm
- net SD_DAT1: track 102.1 -> 70.9 mm, vias 4 -> 2
- net DB2_5V: track 23.2 -> 54.2 mm
- net A0_5V: track 44.7 -> 75.0 mm
- net SD_CLK: track 111.0 -> 81.1 mm, vias 4 -> 2
- net DB4_5V: track 22.4 -> 51.9 mm, vias 0 -> 1
- net MISO_D0: track 111.8 -> 83.1 mm
- net DB3_5V: track 27.6 -> 54.1 mm
- net GND: track 240.0 -> 264.3 mm, vias 17 -> 19
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Other:
- board text added: "Experimental School's Computer Desktop Touch Keyboard V2.0 June 2024 menadue@gmail.com"
- board text removed: "Experimental School's Computer Desktop Touch Keyboard V1.0 May 2024 menadue@gmail.com"
