File: pcbs/touch_keyboard/touch_with_qt/qt_touch1/levelshift.sch (KiCad schematic (older format))
At the start: 8 parts

Commit message: Updates
Parts:
- removed R22, R23, R24, R25: 4k7, Resistor_SMD:R_0805_2012Metric_Pad1.20x1.40mm_HandSolder, symbol Device:R_Small
- removed TR1, TR2, TR3, TR4: Si2302CDS-n-channel, Package_TO_SOT_SMD:SOT-23, symbol New_Library:Si2302CDS-n-channel
- added C12, C13, C14, C15: 100nF, symbol Device:C_Small
- added U2, U3: cd40109, Package_SO:SOP-24_7.5x15.4mm_P1.27mm, symbol ajm:cd40109
- added U4, U5: cd40109, symbol ajm:cd40109
Connections:
- net +3V3: now also C12.1, C13.1, U2.1 (VCC), U3.16 (VDD)
- net +5V: now also C14.1, C15.1, U2.16 (VDD), U3.1 (VCC)
- net GND: now also C12.2, C13.2, C14.2, C15.2, U2.8 (VSS), U3.8 (VSS)
- net RX_3V3: now also U2.3
- net RX_5V: now also U2.4
- net TX_3V3: now also U3.4
- net TX_5V: now also U3.3
- new net DRDY_3V3: U3.5
- new net DRDY_5V: U3.6
- new net MISO_3V3: U2.5
- new net MISO_5V: U2.6
- new net MOSI_3V3: U4.3
- new net MOSI_5V: U4.4
- new net SCK_3v3: U5.3
- new net SCK_5V: U5.4
Other:
- note added: "Shift DOWN\n5V to 3V3"
- note added: "Shift UP\n3V3 to 5V"

Commit message: Updates
Parts:
- C12, C13, C14, C15: footprint (none) -> Capacitor_SMD:C_0805_2012Metric_Pad1.18x1.45mm_HandSolder
- U2: renamed from U5; footprint (none) -> Package_SO:SOP-24_7.5x15.4mm_P1.27mm
- U2: renamed from U4; footprint (none) -> Package_SO:SOP-24_7.5x15.4mm_P1.27mm
- renumbered U2 to U3
Connections:
- net MISO_3V3: now also U3.11; no longer U3.5
- net MISO_5V: now also U3.10; no longer U3.6
- net MOSI_3V3: now also U2.6; no longer U2.3
- net MOSI_5V: now also U2.5; no longer U2.4
- net SCK_3v3: now also U2.10; no longer U2.3
- net SCK_5V: now also U2.11; no longer U2.4
Changed lines of the file:
@@
 F 0 "C14" H 4517 1121 50  0000 L CNN
 F 1 "100nF" H 4517 1030 50  0000 L CNN
-F 2 "" H 4425 1075 50  0001 C CNN
+F 2 "Capacitor_SMD:C_0805_2012Metric_Pad1.18x1.45mm_HandSolder" H 4425 1075 50  0001 C CNN
 F 3 "~" H 4425 1075 50  0001 C CNN
 	1    4425 1075
@@
 F 0 "C15" H 4917 1121 50  0000 L CNN
 F 1 "100nF" H 4917 1030 50  0000 L CNN
-F 2 "" H 4825 1075 50  0001 C CNN
+F 2 "Capacitor_SMD:C_0805_2012Metric_Pad1.18x1.45mm_HandSolder" H 4825 1075 50  0001 C CNN
 F 3 "~" H 4825 1075 50  0001 C CNN
 	1    4825 1075
@@
 F 0 "C12" H 3592 1146 50  0000 L CNN
 F 1 "100nF" H 3592 1055 50  0000 L CNN
-F 2 "" H 3500 1100 50  0001 C CNN
+F 2 "Capacitor_SMD:C_0805_2012Metric_Pad1.18x1.45mm_HandSolder" H 3500 1100 50  0001 C CNN
 F 3 "~" H 3500 1100 50  0001 C CNN
 	1    3500 1100
@@
 F 0 "C13" H 3992 1146 50  0000 L CNN
 F 1 "100nF" H 3992 1055 50  0000 L CNN
-F 2 "" H 3900 1100 50  0001 C CNN
+F 2 "Capacitor_SMD:C_0805_2012Metric_Pad1.18x1.45mm_HandSolder" H 3900 1100 50  0001 C CNN
 F 3 "~" H 3900 1100 50  0001 C CNN
 	1    3900 1100
@@
 SCK_5V
 $Comp
-L ajm:cd40109 U2
-U 2 1 664E659D
+L ajm:cd40109 U3
+U 3 1 664E659D
 P 9800 5575
-F 0 "U2" H 9800 5350 50  0000 C CNN
+F 0 "U3" H 9800 5350 50  0000 C CNN
 F 1 "cd40109" H 9800 5259 50  0000 C CNN
 F 2 "Package_SO:SOP-24_7.5x15.4mm_P1.27mm" H 9600 5875 50  0001 C CNN
 F 3 "" H 9600 5875 50  0001 C CNN
-	2    9800 5575
+	3    9800 5575
 	1    0    0    -1
 $EndComp
@@
 	10100 5575 10450 5575
 $Comp
-L ajm:cd40109 U5
-U 1 1 664E9FC5
+L ajm:cd40109 U2
+U 3 1 664E9FC5
 P 7125 5500
-F 0 "U5" H 7125 5275 50  0000 C CNN
+F 0 "U2" H 7125 5275 50  0000 C CNN
 F 1 "cd40109" H 7125 5184 50  0000 C CNN
-F 2 "" H 6925 5800 50  0001 C CNN
+F 2 "Package_SO:SOP-24_7.5x15.4mm_P1.27mm" H 6925 5800 50  0001 C CNN
 F 3 "" H 6925 5800 50  0001 C CNN
-	1    7125 5500
+	3    7125 5500
 	1    0    0    -1
 $EndComp
 $Comp
-L ajm:cd40109 U4
-U 1 1 664EAA8B
+L ajm:cd40109 U2
+U 2 1 664EAA8B
 P 7125 4825
-F 0 "U4" H 7125 4600 50  0000 C CNN
+F 0 "U2" H 7125 4600 50  0000 C CNN
 F 1 "cd40109" H 7125 4509 50  0000 C CNN
-F 2 "" H 6925 5125 50  0001 C CNN
+F 2 "Package_SO:SOP-24_7.5x15.4mm_P1.27mm" H 6925 5125 50  0001 C CNN
 F 3 "" H 6925 5125 50  0001 C CNN
-	1    7125 4825
+	2    7125 4825
 	1    0    0    -1
 $EndComp

Commit message: Updates
Parts:
- added unit 4 of U2
- added unit 4 of U3
- added U4: cd40109, Package_SO:SOP-24_7.5x15.4mm_P1.27mm, symbol ajm:cd40109
Connections:
- net +3V3: now also U2.2, U2.7, U2.9, U2.15, U4.16 (VDD)
- net +5V: now also U3.2, U3.7, U3.9, U3.15, U4.1 (VCC), U4.15, U4.2, U4.7, U4.9
- net GND: now also U4.10, U4.14, U4.3, U4.8 (VSS)
- net SCK_3v3 renamed SCK_3V3
- new net DBG_CLK3V3: U4.5
- new net DBG_CLK_5V: U4.6
- new net DBG_DATA_3V3: U3.13
- new net DBG_DATA_5V: U3.14
- new net WS_3V3: U2.14
- new net WS_5V: U2.13
Other:
- moved on the sheet: C12, C13, C14, C15, U2A, U2B, U2C, U2E, U3A, U3B, U3C, U3E

Commit message: Updates
Parts:
- U2, U3, U4: footprint Package_SO:SOP-24_7.5x15.4mm_P1.27mm -> Package_SO:SOIC-16W_7.5x10.3mm_P1.27mm
Changed lines of the file:
@@
 F 0 "U2" H 3925 3925 50  0000 C CNN
 F 1 "cd40109" H 3925 3834 50  0000 C CNN
-F 2 "Package_SO:SOP-24_7.5x15.4mm_P1.27mm" H 3725 4450 50  0001 C CNN
+F 2 "Package_SO:SOIC-16W_7.5x10.3mm_P1.27mm" H 3725 4450 50  0001 C CNN
 F 3 "" H 3725 4450 50  0001 C CNN
 	1    3925 4150
@@
 F 0 "U2" H 4103 1846 50  0000 L CNN
 F 1 "cd40109" H 4103 1755 50  0000 L CNN
-F 2 "Package_SO:SOP-24_7.5x15.4mm_P1.27mm" H 3525 2125 50  0001 C CNN
+F 2 "Package_SO:SOIC-16W_7.5x10.3mm_P1.27mm" H 3525 2125 50  0001 C CNN
 F 3 "" H 3525 2125 50  0001 C CNN
 	5    3725 1825
@@
 F 0 "U3" H 7575 3075 50  0000 C CNN
 F 1 "cd40109" H 7650 3000 50  0000 C CNN
-F 2 "Package_SO:SOP-24_7.5x15.4mm_P1.27mm" H 7825 3150 50  0001 C CNN
+F 2 "Package_SO:SOIC-16W_7.5x10.3mm_P1.27mm" H 7825 3150 50  0001 C CNN
 F 3 "" H 7825 3150 50  0001 C CNN
 	1    8025 2850
@@
 F 0 "U3" H 7828 1796 50  0000 L CNN
 F 1 "cd40109" H 7828 1705 50  0000 L CNN
-F 2 "Package_SO:SOP-24_7.5x15.4mm_P1.27mm" H 7250 2075 50  0001 C CNN
+F 2 "Package_SO:SOIC-16W_7.5x10.3mm_P1.27mm" H 7250 2075 50  0001 C CNN
 F 3 "" H 7250 2075 50  0001 C CNN
 	5    7450 1775
@@
 F 0 "U3" H 7550 3575 50  0000 C CNN
 F 1 "cd40109" H 7625 3500 50  0000 C CNN
-F 2 "Package_SO:SOP-24_7.5x15.4mm_P1.27mm" H 7825 3675 50  0001 C CNN
+F 2 "Package_SO:SOIC-16W_7.5x10.3mm_P1.27mm" H 7825 3675 50  0001 C CNN
 F 3 "" H 7825 3675 50  0001 C CNN
 	2    8025 3375
@@
 F 0 "U3" H 7525 4150 50  0000 C CNN
 F 1 "cd40109" H 7600 4075 50  0000 C CNN
-F 2 "Package_SO:SOP-24_7.5x15.4mm_P1.27mm" H 7825 4225 50  0001 C CNN
+F 2 "Package_SO:SOIC-16W_7.5x10.3mm_P1.27mm" H 7825 4225 50  0001 C CNN
 F 3 "" H 7825 4225 50  0001 C CNN
 	3    8025 3925
@@
 F 0 "U2" H 3950 5250 50  0000 C CNN
 F 1 "cd40109" H 3950 5159 50  0000 C CNN
-F 2 "Package_SO:SOP-24_7.5x15.4mm_P1.27mm" H 3750 5775 50  0001 C CNN
+F 2 "Package_SO:SOIC-16W_7.5x10.3mm_P1.27mm" H 3750 5775 50  0001 C CNN
 F 3 "" H 3750 5775 50  0001 C CNN
 	3    3950 5475
@@
 F 0 "U2" H 3950 4575 50  0000 C CNN
 F 1 "cd40109" H 3950 4484 50  0000 C CNN
-F 2 "Package_SO:SOP-24_7.5x15.4mm_P1.27mm" H 3750 5100 50  0001 C CNN
+F 2 "Package_SO:SOIC-16W_7.5x10.3mm_P1.27mm" H 3750 5100 50  0001 C CNN
 F 3 "" H 3750 5100 50  0001 C CNN
 	2    3950 4800
@@
 F 0 "U3" H 7500 4675 50  0000 C CNN
 F 1 "cd40109" H 7600 4600 50  0000 C CNN
-F 2 "Package_SO:SOP-24_7.5x15.4mm_P1.27mm" H 7825 4800 50  0001 C CNN
+F 2 "Package_SO:SOIC-16W_7.5x10.3mm_P1.27mm" H 7825 4800 50  0001 C CNN
 F 3 "" H 7825 4800 50  0001 C CNN
 	4    8025 4500
@@
 F 0 "U4" H 8978 1796 50  0000 L CNN
 F 1 "cd40109" H 8978 1705 50  0000 L CNN
-F 2 "Package_SO:SOP-24_7.5x15.4mm_P1.27mm" H 8400 2075 50  0001 C CNN
+F 2 "Package_SO:SOIC-16W_7.5x10.3mm_P1.27mm" H 8400 2075 50  0001 C CNN
 F 3 "" H 8400 2075 50  0001 C CNN
 	5    8600 1775
@@
 F 0 "U4" H 7500 5250 50  0000 C CNN
 F 1 "cd40109" H 7600 5175 50  0000 C CNN
-F 2 "Package_SO:SOP-24_7.5x15.4mm_P1.27mm" H 7825 5375 50  0001 C CNN
+F 2 "Package_SO:SOIC-16W_7.5x10.3mm_P1.27mm" H 7825 5375 50  0001 C CNN
 F 3 "" H 7825 5375 50  0001 C CNN
 	2    8025 5075
@@
 F 0 "U2" H 3950 5875 50  0000 C CNN
 F 1 "cd40109" H 3950 5784 50  0000 C CNN
-F 2 "Package_SO:SOP-24_7.5x15.4mm_P1.27mm" H 3750 6400 50  0001 C CNN
+F 2 "Package_SO:SOIC-16W_7.5x10.3mm_P1.27mm" H 3750 6400 50  0001 C CNN
 F 3 "" H 3750 6400 50  0001 C CNN
 	4    3950 6100
@@
 F 0 "U4" H 7500 5700 50  0000 C CNN
 F 1 "cd40109" H 7600 5625 50  0000 C CNN
-F 2 "Package_SO:SOP-24_7.5x15.4mm_P1.27mm" H 7825 5825 50  0001 C CNN
+F 2 "Package_SO:SOIC-16W_7.5x10.3mm_P1.27mm" H 7825 5825 50  0001 C CNN
 F 3 "" H 7825 5825 50  0001 C CNN
 	1    8025 5525
@@
 F 0 "U4" H 7500 6075 50  0000 C CNN
 F 1 "cd40109" H 7600 6000 50  0000 C CNN
-F 2 "Package_SO:SOP-24_7.5x15.4mm_P1.27mm" H 7825 6200 50  0001 C CNN
+F 2 "Package_SO:SOIC-16W_7.5x10.3mm_P1.27mm" H 7825 6200 50  0001 C CNN
 F 3 "" H 7825 6200 50  0001 C CNN
 	3    8025 5900
@@
 F 0 "U4" H 7500 6450 50  0000 C CNN
 F 1 "cd40109" H 7600 6375 50  0000 C CNN
-F 2 "Package_SO:SOP-24_7.5x15.4mm_P1.27mm" H 7825 6575 50  0001 C CNN
+F 2 "Package_SO:SOIC-16W_7.5x10.3mm_P1.27mm" H 7825 6575 50  0001 C CNN
 F 3 "" H 7825 6575 50  0001 C CNN
 	4    8025 6275
