File: pcbs/touch_keyboard/touch_with_qt/qt_touch1/keys.sch (KiCad schematic (older format))
At the start: 32 parts

Commit message: Updates
Parts:
- removed TP1, TP10, TP11, TP12, TP13, TP14, TP15, TP16, TP17, TP18, TP19, TP2, TP20, TP21, TP22, TP23, TP24, TP25, TP26, TP27, TP28, TP29, TP3, TP30, TP31, TP32, TP4, TP5, TP6, TP7, TP8, TP9: TestPoint, ajm_kicad:qt_touch_12_x_12, symbol Connector:TestPoint
- added TP1, TP10, TP11, TP12, TP13, TP14, TP15, TP16, TP17, TP18, TP19, TP2, TP20, TP21, TP22, TP23, TP24, TP25, TP26, TP27, TP28, TP3, TP4, TP5, TP6, TP7, TP8, TP9: Touchpad_qt, ajm_kicad:qt_touch_12_x_12, symbol ajm:Touchpad_qt
Connections:
- new net X7: TP10.X, TP16.X, TP2.X, TP22.X

Commit message: Updates
Connections:
- net X0: now also TP5.X
- net X1: now also TP15.X, TP9.X
- net X2: now also TP12.X, TP20.X, TP4.X
- net X3: now also TP1.X
- net X4: now also TP13.X, TP21.X, TP25.X, TP7.X
- net X5: now also TP11.X, TP18.X, TP23.X, TP27.X, TP3.X
- net X6: now also TP14.X, TP19.X, TP24.X, TP6.X
- net X7: now also TP26.X
- net Y0: now also TP10.Y, TP11.Y, TP2.Y, TP3.Y, TP6.Y, TP7.Y
- net Y1: now also TP13.Y, TP14.Y, TP16.Y, TP18.Y, TP19.Y, TP21.Y, TP22.Y, TP23.Y
- net Y2: now also TP25.Y, TP26.Y, TP27.Y, TP28.Y
- net Y3: now also TP1.Y, TP4.Y, TP8.Y
- net Y4: now also TP12.Y, TP5.Y, TP9.Y
- net Y5: now also TP15.Y, TP17.Y, TP20.Y
- net at TP8.X: now also TP17.X

Commit message: Updates
Connections:
- net X4: now also TP28.X
- net Y2: now also TP24.Y
Changed lines of the file:
@@
 Connection ~ 5875 3350
-Wire Wire Line
-	7300 3350 8600 3350
 Wire Wire Line
 	8600 3350 8600 3800
@@
 	8975 1925 8625 1925
 Wire Wire Line
-	8975 1925 8975 3125
+	8975 1925 8975 2450
 Wire Wire Line
 	8975 3125 8675 3125
@@
 	4300 6425 4300 5700
 Connection ~ 3500 6425
+Wire Wire Line
+	8075 2450 8975 2450
+Connection ~ 8975 2450
+Wire Wire Line
+	8975 2450 8975 3125
+Wire Wire Line
+	7225 3350 8600 3350
+Connection ~ 7225 3350
 $EndSCHEMATC

Commit message: Updates
Connections:
- net X3: now also TP17.X, TP8.X
Changed lines of the file:
@@
 	1300 4225 1075 4225
 Wire Wire Line
-	1075 4225 1075 5100
-Wire Wire Line
-	1100 4575 2475 4575
+	1075 4225 1075 4575
 Wire Wire Line
 	2475 4575 2475 5100
@@
 	7225 3350 8600 3350
 Connection ~ 7225 3350
+Wire Wire Line
+	1075 4575 2475 4575
+Connection ~ 1075 4575
+Wire Wire Line
+	1075 4575 1075 5100
 $EndSCHEMATC

Commit message: Updates
Connections:
- net X0: now also TP1.X, TP14.X, TP2.X, TP28.X
- net X1: now also TP13.X
- net X2: now also TP18.X
- net X3: no longer TP1.X
- net X4: now also TP3.X; no longer TP13.X, TP28.X
- net X5: no longer TP18.X, TP3.X
- net X6: no longer TP14.X
- net X7: no longer TP2.X
Changed lines of the file:
@@
-$EndComp
-$Comp
-L ajm:Touchpad_qt TP3
-U 1 1 664ABAAE
-P 1925 2800
-F 0 "TP3" H 2000 2865 50  0000 C CNN
-F 1 "Touchpad_qt" H 2000 2774 50  0000 C CNN
-F 2 "ajm_kicad:qt_touch_12_x_12" H 1925 2800 50  0001 C CNN
-F 3 "" H 1925 2800 50  0001 C CNN
-	1    1925 2800
-	1    0    0    -1
 $EndComp
 $Comp
@@
 Y5
 Wire Wire Line
-	925  1875 1475 1875
-Wire Wire Line
-	1475 1875 1475 1275
-Wire Wire Line
-	1475 1275 3200 1275
+	925  1875 1150 1875
 Wire Wire Line
 	3200 1275 3200 1875
-Connection ~ 1475 1875
 Wire Wire Line
 	3200 1275 5025 1275
@@
 Wire Wire Line
 	2375 1975 2375 2450
-Wire Wire Line
-	2375 1975 4550 1975
-Wire Wire Line
-	4550 1975 4550 2475
 Connection ~ 2375 1975
 Wire Wire Line
-	4550 1975 4950 1975
-Wire Wire Line
 	4950 1975 4950 2075
 Wire Wire Line
@@
 Wire Wire Line
 	5750 2075 5750 2475
-Connection ~ 4550 1975
 Wire Wire Line
 	5750 2075 7125 2075
@@
 Wire Wire Line
 	3250 2625 3250 3075
-Connection ~ 1525 2625
-Wire Wire Line
-	1525 2625 1525 3050
-Wire Wire Line
-	3250 2625 5100 2625
-Wire Wire Line
-	5100 2625 5100 3125
 Connection ~ 3250 2625
 Wire Wire Line
-	5100 2625 6400 2625
-Wire Wire Line
 	6400 2625 6400 3125
-Connection ~ 5100 2625
 Wire Wire Line
 	6400 2625 7725 2625
@@
 	925  2175 1375 2175
 Wire Wire Line
-	1375 2175 1375 3775
+	1375 2175 1375 3050
 Wire Wire Line
 	1375 3775 2350 3775
 Wire Wire Line
 	2350 3775 2350 3350
-Wire Wire Line
-	2350 3350 4400 3350
-Wire Wire Line
-	4400 3350 4400 3800
 Connection ~ 2350 3775
 Wire Wire Line
 	2350 3775 2450 3775
 Wire Wire Line
-	4400 3350 5875 3350
-Wire Wire Line
 	5875 3350 5875 3825
-Connection ~ 4400 3350
 Wire Wire Line
 	5875 3350 7225 3350
@@
 Connection ~ 5875 3350
 Wire Wire Line
-	8600 3350 8600 3800
-Wire Wire Line
 	925  2275 1300 2275
 Wire Wire Line
@@
 	1075 4075 775  4075
 Wire Wire Line
-	775  4075 775  7175
+	775  4075 775  5100
 Wire Wire Line
 	775  7175 1750 7175
@@
 	8975 2450 8975 3125
 Wire Wire Line
-	7225 3350 8600 3350
-Connection ~ 7225 3350
-Wire Wire Line
 	1075 4575 2475 4575
-Connection ~ 1075 4575
-Wire Wire Line
-	1075 4575 1075 5100
+Wire Wire Line
+	1075 5100 775  5100
+Connection ~ 775  5100
+Wire Wire Line
+	775  5100 775  7175
+Text GLabel 8550 3800 0    50   Input ~ 0
+X0
+Wire Wire Line
+	8550 3800 8600 3800
+Wire Wire Line
+	2375 1975 4950 1975
+Text GLabel 4475 2475 0    50   Input ~ 0
+X0
+Wire Wire Line
+	4475 2475 4550 2475
+Wire Wire Line
+	3250 2625 6400 2625
+Text GLabel 5000 3125 0    50   Input ~ 0
+X2
+Wire Wire Line
+	5000 3125 5100 3125
+Wire Wire Line
+	2350 3350 5875 3350
+Text GLabel 4400 3800 0    50   Input ~ 0
+X1
+Wire Wire Line
+	1150 1275 1150 1875
+Wire Wire Line
+	1150 1275 3200 1275
+Text GLabel 1400 1875 0    50   Input ~ 0
+X0
+Wire Wire Line
+	1400 1875 1475 1875
+$Comp
+L ajm:Touchpad_qt TP3
+U 1 1 664ABAAE
+P 1925 2800
+F 0 "TP3" H 2000 2865 50  0000 C CNN
+F 1 "Touchpad_qt" H 2000 2774 50  0000 C CNN
+F 2 "ajm_kicad:qt_touch_12_x_12" H 1925 2800 50  0001 C CNN
+F 3 "" H 1925 2800 50  0001 C CNN
+	1    1925 2800
+	1    0    0    -1
+$EndComp
+Wire Wire Line
+	1525 3050 1375 3050
+Connection ~ 1375 3050
+Wire Wire Line
+	1375 3050 1375 3775
 $EndSCHEMATC

Commit message: Updates
Parts:
- TP1: value Touchpad_qt -> A
- TP10: value Touchpad_qt -> LOAD ADDR
- TP11: value Touchpad_qt -> INCR ADDR
- TP12: value Touchpad_qt -> STOP
- TP13: value Touchpad_qt -> 7
- TP14: value Touchpad_qt -> 1
- TP15: value Touchpad_qt -> RELOAD
- TP16: value Touchpad_qt -> CLEAR
- TP17: value Touchpad_qt -> DUMP
- TP18: value Touchpad_qt -> 4
- TP19: value Touchpad_qt -> 2
- TP2: value Touchpad_qt -> LOAD IAR
- TP20: value Touchpad_qt -> CHECK
- TP21: value Touchpad_qt -> 8
- TP22: value Touchpad_qt -> MINUS
- TP23: value Touchpad_qt -> 5
- TP24: value Touchpad_qt -> 3
- TP25: value Touchpad_qt -> 9
- TP26: value Touchpad_qt -> DOT
- TP27: value Touchpad_qt -> 6
- TP28: value Touchpad_qt -> 0
- TP3: value Touchpad_qt -> DECR ADDR
- TP4: value Touchpad_qt -> B
- TP5: value Touchpad_qt -> KI RESET
- TP6: value Touchpad_qt -> LOAD STORE
- TP7: value Touchpad_qt -> NORM RESET
- TP8: value Touchpad_qt -> RUN
- TP9: value Touchpad_qt -> C
Connections:
- net X2: now also TP22.Y, TP7.X
- net X3: now also TP16.X
- net X4: no longer TP7.X
- net X7: no longer TP16.X
- net Y0: now also TP1.Y, TP4.Y, TP8.Y; no longer TP10.Y, TP11.Y, TP2.Y, TP3.Y, TP6.Y, TP7.Y
- net Y1: now also TP24.Y, TP25.Y, TP26.Y, TP27.Y, TP28.Y; no longer TP13.Y, TP14.Y, TP16.Y, TP18.Y, TP19.Y, TP21.Y, TP22.Y, TP23.Y
- net Y2: now also TP13.Y, TP14.Y, TP16.Y, TP18.Y, TP19.Y, TP21.Y, TP23.Y; no longer TP24.Y, TP25.Y, TP26.Y, TP27.Y, TP28.Y
- net Y3: now also TP10.Y, TP11.Y, TP2.Y, TP3.Y, TP6.Y, TP7.Y; no longer TP1.Y, TP4.Y, TP8.Y
Other:
- moved on the sheet: TP1, TP12, TP14, TP15, TP17, TP20, TP22, TP4, TP5, TP8, TP9

Commit message: Updates
Connections:
- net X2: no longer TP22.Y
- net Y2: now also TP22.Y
Changed lines of the file:
@@
 X7
 Text GLabel 7325 1925 2    50   Input ~ 0
-X2
+Y2
 $EndSCHEMATC
