File: pcbs/touch_keyboard/touch_with_qt/qt_touch1/qt_touch1.kicad_pcb (KiCad board)
At the start: 2 copper layers, 229 x 104.5 mm, 69 parts, among them J1 Conn_01x05_Female, U1 74HC165, U2 74HC165, U3 74HC165, U4 74HC165

Commit message: Updates
Parts:
- removed J1: Conn_01x05_Female, Connector_PinHeader_2.54mm:PinHeader_1x05_P2.54mm_Vertical_SMD_Pin1Left
- removed LOAD ADDR: TestPoint, ajm_kicad:ESC_KB_Pad_half_size
- removed LOAD IAR: TestPoint, ajm_kicad:ESC_KB_Pad_half_size
- removed R22, R23, R24, R25, R26, R27, R28, R29, R30, R31, R32: 10M, Resistor_SMD:R_0805_2012Metric_Pad1.20x1.40mm_HandSolder
- removed TP29, TP31: TestPoint, ajm_kicad:ESC_KB_Pad_half_size
- removed U4: 74HC165, Package_SO:SO-16_3.9x9.9mm_P1.27mm
- added C10: C_Small, ajm_kicad:qt_touch_12_x_12, F.Cu at (268.9, 185.9)
- added C11: C_Small, ajm_kicad:qt_touch_12_x_12, F.Cu at (232.8, 190.5)
- added C5: C_Small, ajm_kicad:qt_touch_12_x_12, F.Cu at (207.2, 190.5)
- added C6: C_Small, ajm_kicad:qt_touch_12_x_12, F.Cu at (221.5, 177.7)
- added C7: C_Small, ajm_kicad:qt_touch_12_x_12, F.Cu at (241.4, 164.9)
- added C8: C_Small, ajm_kicad:qt_touch_12_x_12, F.Cu at (220.0, 190.5)
- added C9: C_Small, ajm_kicad:qt_touch_12_x_12, F.Cu at (215.8, 164.9)
- added TP16: Touchpad_qt, ajm_kicad:qt_touch_12_x_12, F.Cu at (58.6, 62.1)
- added TP26: Touchpad_qt, ajm_kicad:qt_touch_12_x_12, F.Cu at (271.3, 118.7)
- added TP28: Touchpad_qt, ajm_kicad:qt_touch_12_x_12, F.Cu at (271.3, 131.5)
- added TP8: Touchpad_qt, ajm_kicad:qt_touch_12_x_12, F.Cu at (194.3, 144.3)
- added Y1: 16MHz, Crystal:Crystal_SMD_HC49-SD_HandSoldering, F.Cu at (198.6, 161.6)
- C1, C2: value 100nF -> 20pF; footprint Capacitor_SMD:C_0805_2012Metric_Pad1.18x1.45mm_HandSolder -> ajm_kicad:qt_touch_12_x_12; moved to F.Cu
- C3, C4: value 100nF -> C_Small; footprint Capacitor_SMD:C_0805_2012Metric_Pad1.18x1.45mm_HandSolder -> ajm_kicad:qt_touch_12_x_12; moved to F.Cu
- R1: value 10M -> 4k7; moved to F.Cu
- R10, R11, R12, R13, R14, R15, R16, R17, R18, R19, R2, R20, R21, R3, R4, R5, R6, R7, R8, R9: value 10M -> R_Small; moved to F.Cu
- TP1, TP10, TP11, TP12, TP13, TP14, TP15, TP17, TP18, TP19, TP2, TP20, TP21, TP22, TP23, TP24, TP25, TP27, TP3, TP4, TP5, TP6, TP7, TP9: value TestPoint -> Touchpad_qt; footprint ajm_kicad:ESC_KB_Pad_half_size -> ajm_kicad:qt_touch_12_x_12
- U1: value 74HC165 -> QT1481; footprint Package_SO:SO-16_3.9x9.9mm_P1.27mm -> Package_QFP:LQFP-44_10x10mm_P0.8mm; moved to F.Cu
- U2, U3: value 74HC165 -> cd40109; footprint Package_SO:SO-16_3.9x9.9mm_P1.27mm -> Package_SO:SOP-24_7.5x15.4mm_P1.27mm; moved to F.Cu
- moved U2 244.5 mm to (309.8, 107.9)
- moved R10 222.0 mm to (255.9, 174.7)
- moved R14 215.4 mm to (241.6, 185.6)
- moved R12 212.4 mm to (241.6, 188.5)
- moved R16 209.6 mm to (250.2, 162.9)
- moved R8 201.7 mm to (246.3, 188.5), turned to 0 degrees
- moved C4 185.9 mm to (228.6, 164.9), turned to 0 degrees
- moved U3 184.8 mm to (297.0, 107.9)
- moved TP27 175.2 mm to (258.5, 144.3)
- moved TP23 174.9 mm to (271.3, 105.8)
- moved TP14 171.4 mm to (232.8, 118.7)
- moved R4 165.3 mm to (195.0, 193.4), turned to 0 degrees
- moved R2 161.9 mm to (190.3, 196.3), turned to 0 degrees
- moved TP12 157.0 mm to (207.2, 144.3)
- moved R17 154.2 mm to (250.2, 168.8), turned to 0 degrees
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Connections:
- R1 pad 1: GND -> +5V
- R1 pad 2: Net-(R1-Pad2) -> (no net)
- R10 pad 1: GND -> Net-(R10-Pad1)
- R10 pad 2: Net-(R10-Pad2) -> (no net)
- R11 pad 1: GND -> Net-(R11-Pad1)
- R11 pad 2: Net-(R11-Pad2) -> (no net)
- R12 pad 1: GND -> Net-(R12-Pad1)
- R12 pad 2: Net-(R12-Pad2) -> (no net)
- R13 pad 1: GND -> Net-(R13-Pad1)
- R13 pad 2: Net-(R13-Pad2) -> (no net)
- R14 pad 1: GND -> Net-(R14-Pad1)
- R14 pad 2: Net-(R14-Pad2) -> (no net)
- R15 pad 1: GND -> Net-(R15-Pad1)
- R15 pad 2: Net-(R15-Pad2) -> (no net)
- R16 pad 1: GND -> Net-(C6-Pad1)
- R16 pad 2: Net-(R16-Pad2) -> (no net)
- R17 pad 1: GND -> Net-(C7-Pad1)
- R17 pad 2: Net-(R17-Pad2) -> (no net)
- R18 pad 1: GND -> Net-(C8-Pad1)
- R18 pad 2: Net-(R18-Pad2) -> (no net)
- R19 pad 1: GND -> Net-(C9-Pad1)
- R19 pad 2: Net-(R19-Pad2) -> (no net)
- R2 pad 1: GND -> Net-(C11-Pad2)
- R20 pad 1: GND -> Net-(C10-Pad1)
- R20 pad 2: Net-(R20-Pad2) -> (no net)
- R21 pad 1: GND -> Net-(C11-Pad1)
- R21 pad 2: Net-(R21-Pad2) -> (no net)
- R3 pad 1: GND -> Net-(C10-Pad2)
- R3 pad 2: Net-(R3-Pad2) -> Net-(R2-Pad2)
- R4 pad 1: GND -> Net-(C9-Pad2)
- R4 pad 2: Net-(R4-Pad2) -> Net-(R2-Pad2)
- R5 pad 1: GND -> Net-(C8-Pad2)
- R5 pad 2: Net-(R5-Pad2) -> Net-(R2-Pad2)
- R6 pad 1: GND -> Net-(C7-Pad2)
- R6 pad 2: Net-(R6-Pad2) -> Net-(R2-Pad2)
- R7 pad 1: GND -> Net-(R7-Pad1)
- R7 pad 2: Net-(R7-Pad2) -> X7
- R8 pad 1: GND -> Net-(R8-Pad1)
- R8 pad 2: Net-(R8-Pad2) -> (no net)
- R9 pad 1: GND -> Net-(C6-Pad2)
- R9 pad 2: Net-(R9-Pad2) -> Net-(R2-Pad2)
- U1 pad 1: LOAD -> (no net)
- U1 pad 10: SERDAT_OUT_2 -> TX_5V
- U1 pad 11: Net-(R1-Pad2) -> (no net)
- U1 pad 12: Net-(R3-Pad2) -> Net-(R2-Pad2)
- U1 pad 13: Net-(R5-Pad2) -> Net-(C9-Pad1)
- U1 pad 14: Net-(R7-Pad2) -> Net-(C8-Pad1)
- U1 pad 15: GND -> Net-(C7-Pad1)
- U1 pad 16: +3V3 -> Net-(C6-Pad1)
- U1 pad 2: CLK -> MISO_5V
- U1 pad 3: Net-(R9-Pad2) -> (no net)
- U1 pad 4: Net-(R11-Pad2) -> Net-(C3-Pad1)
- U1 pad 5: Net-(R13-Pad2) -> Net-(C3-Pad1)
- U1 pad 6: Net-(R15-Pad2) -> GND
- U1 pad 7: (no net) -> Net-(C2-Pad1)
- U1 pad 8: GND -> Net-(C1-Pad1)
- U1 pad 9: SERDAT_OUT_3 -> RX_5V
- U2 pad 1: LOAD -> +3V3
- U2 pad 11: Net-(R2-Pad2) -> (no net)
- U2 pad 12: Net-(R4-Pad2) -> (no net)
- U2 pad 13: Net-(R6-Pad2) -> (no net)
- U2 pad 14: Net-(R8-Pad2) -> (no net)
- U2 pad 15: GND -> (no net)
- U2 pad 16: +3V3 -> +5V
- U2 pad 2: CLK -> (no net)
- U2 pad 3: Net-(R10-Pad2) -> (no net)
- U2 pad 4: Net-(R12-Pad2) -> RX_5V
- U2 pad 5: Net-(R14-Pad2) -> (no net)
- U2 pad 6: Net-(R16-Pad2) -> MISO_5V
- U2 pad 9: SERDAT_OUT_1 -> (no net)
- U3 pad 1: LOAD -> +5V
- U3 pad 10: SERDAT_OUT_1 -> (no net)
- U3 pad 11: Net-(R17-Pad2) -> (no net)
- U3 pad 12: Net-(R19-Pad2) -> (no net)
- U3 pad 13: Net-(R21-Pad2) -> (no net)
- U3 pad 14: Net-(R23-Pad2) -> (no net)
- U3 pad 15: GND -> (no net)
- U3 pad 2: CLK -> (no net)
- U3 pad 3: Net-(R25-Pad2) -> TX_5V
- U3 pad 4: Net-(R27-Pad2) -> (no net)
- U3 pad 5: Net-(R29-Pad2) -> (no net)
- U3 pad 6: Net-(R31-Pad2) -> DRDY_5V
- U3 pad 9: SERDAT_OUT_2 -> (no net)
Routing:
- net Net-(TP4-PadX): track 0.00 -> 654.0 mm, vias 0 -> 20
- net +3V3: track 375.9 -> 0.00 mm, vias 11 -> 0
- net CLK: track 210.0 -> 0.00 mm, vias 6 -> 0
- net Net-(R13-Pad2): track 68.1 -> 0.00 mm, vias 3 -> 0
- net X7: track 0.00 -> 44.6 mm, vias 0 -> 3
- net Net-(R8-Pad2): track 44.6 -> 0.00 mm, vias 3 -> 0
- net Net-(TP4-PadY): track 0.00 -> 35.2 mm, vias 0 -> 3
- net Net-(R16-Pad2): track 35.2 -> 0.00 mm, vias 3 -> 0
- net Net-(TP7-PadY): track 0.00 -> 30.0 mm, vias 0 -> 1
- net Net-(R24-Pad2): track 30.0 -> 0.00 mm, vias 1 -> 0

Commit message: Updates
Parts:
- added C12: 100nF, Capacitor_SMD:C_0805_2012Metric_Pad1.18x1.45mm_HandSolder, B.Cu at (75.5, 139.7)
- added C13: 100nF, Capacitor_SMD:C_0805_2012Metric_Pad1.18x1.45mm_HandSolder, B.Cu at (38.6, 117.7)
- added C14: 100nF, Capacitor_SMD:C_0805_2012Metric_Pad1.18x1.45mm_HandSolder, B.Cu at (73.7, 118.8)
- added C15: 100nF, Capacitor_SMD:C_0805_2012Metric_Pad1.18x1.45mm_HandSolder, B.Cu at (60.6, 118.5)
- added C16: C_Small, Capacitor_SMD:C_0805_2012Metric_Pad1.18x1.45mm_HandSolder, B.Cu at (160.1, 22.4)
- added C17: C_Small, Capacitor_SMD:C_0805_2012Metric_Pad1.18x1.45mm_HandSolder, B.Cu at (171.5, 21.2)
- added D1: LED, LED_SMD:LED_0805_2012Metric_Pad1.15x1.40mm_HandSolder, B.Cu at (190.1, 139.5)
- added D2: D, LED_SMD:LED_0805_2012Metric_Pad1.15x1.40mm_HandSolder, F.Cu at (74.9, 42.1)
- added J1: Conn_01x12_Female, Connector_PinSocket_2.54mm:PinSocket_1x12_P2.54mm_Vertical_SMD_Pin1Left, B.Cu at (34.6, 88.7)
- added R22: R_Small, Resistor_SMD:R_0805_2012Metric_Pad1.20x1.40mm_HandSolder, F.Cu at (79.7, 42.1)
- C1, C10, C11, C2, C3, C4, C5, C6, C7, C8, C9: footprint ajm_kicad:qt_touch_12_x_12 -> Capacitor_SMD:C_0805_2012Metric_Pad1.18x1.45mm_HandSolder; moved to B.Cu
- R1, R10, R11, R12, R13, R14, R15, R16, R17, R18, R19, R2, R20, R21, R3, R4, R5, R6, R7, R8, R9, U1, U2, U3, Y1: moved to B.Cu
- moved U2 252.1 mm to (58.7, 130.8), turned to 180 degrees
- moved U3 223.9 mm to (74.1, 129.4), turned to 180 degrees
- moved TP2 187.0 mm to (58.9, 62.7)
- moved TP11 159.5 mm to (73.9, 92.7)
- moved TP10 156.4 mm to (73.9, 62.7)
- moved TP7 153.6 mm to (66.4, 107.2)
- moved TP23 153.0 mm to (118.9, 92.7)
- moved TP22 150.4 mm to (118.9, 62.7)
- moved TP19 149.9 mm to (111.2, 77.7)
- moved TP26 148.4 mm to (133.9, 62.7)
- moved TP6 146.6 mm to (66.4, 77.7)
- moved TP18 144.1 mm to (103.9, 92.9)
- moved TP14 142.4 mm to (96.4, 77.7)
- moved TP3 137.9 mm to (58.9, 92.7)
- moved TP24 136.6 mm to (126.4, 77.7)
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Connections:
- R1 pad 2: (no net) -> Net-(D1-Pad1)
- R10 pad 2: (no net) -> X6
- R12 pad 2: (no net) -> X5
- R13 pad 2: (no net) -> X1
- R14 pad 2: (no net) -> X4
- R15 pad 2: (no net) -> X0
- R16 pad 2: (no net) -> Y0
- R17 pad 2: (no net) -> Y1
- R18 pad 2: (no net) -> Y2
- R19 pad 2: (no net) -> Y3
- R20 pad 2: (no net) -> Y4
- R21 pad 2: (no net) -> Y5
- R8 pad 2: (no net) -> X3
- TP1 pad X: Net-(TP1-PadX) -> X3
- TP1 pad Y: Net-(TP1-PadY) -> Y3
- TP10 pad Y: Net-(TP10-PadY) -> Y0
- TP11 pad X: Net-(TP11-PadX) -> X5
- TP11 pad Y: Net-(TP11-PadY) -> Y0
- TP12 pad X: Net-(TP12-PadX) -> X2
- TP12 pad Y: Net-(TP12-PadY) -> Y4
- TP13 pad X: Net-(TP13-PadX) -> X4
- TP13 pad Y: Net-(TP13-PadY) -> Y1
- TP14 pad X: Net-(TP14-PadX) -> X6
- TP14 pad Y: Net-(TP14-PadY) -> Y1
- TP15 pad X: Net-(TP15-PadX) -> X1
- TP15 pad Y: Net-(TP15-PadY) -> Y5
- TP16 pad Y: Net-(TP16-PadY) -> Y1
- TP17 pad Y: Net-(TP17-PadY) -> Y5
- TP18 pad X: Net-(TP18-PadX) -> X5
- TP18 pad Y: Net-(TP18-PadY) -> Y1
- TP19 pad X: Net-(TP19-PadX) -> X6
- TP19 pad Y: Net-(TP19-PadY) -> Y1
- TP2 pad Y: Net-(TP2-PadY) -> Y0
- TP20 pad X: Net-(TP20-PadX) -> X2
- TP20 pad Y: Net-(TP20-PadY) -> Y5
- TP21 pad X: Net-(TP21-PadX) -> X4
- TP21 pad Y: Net-(TP21-PadY) -> Y1
- TP22 pad Y: Net-(TP22-PadY) -> Y1
- TP23 pad X: Net-(TP23-PadX) -> X5
- TP23 pad Y: Net-(TP23-PadY) -> Y1
- TP24 pad X: Net-(TP24-PadX) -> X6
- TP25 pad X: Net-(TP25-PadX) -> X4
- TP25 pad Y: Net-(TP25-PadY) -> Y2
- TP26 pad X: Net-(TP26-PadX) -> X7
- TP26 pad Y: Net-(TP26-PadY) -> Y2
- TP27 pad X: Net-(TP27-PadX) -> X5
- TP27 pad Y: Net-(TP27-PadY) -> Y2
- TP28 pad Y: Net-(TP28-PadY) -> Y2
- TP3 pad X: Net-(TP3-PadX) -> X5
- TP3 pad Y: Net-(TP3-PadY) -> Y0
- TP4 pad X: Net-(TP4-PadX) -> X2
- TP4 pad Y: Net-(TP4-PadY) -> Y3
- TP5 pad X: Net-(TP5-PadX) -> X0
- TP5 pad Y: Net-(TP5-PadY) -> Y4
- TP6 pad X: Net-(TP6-PadX) -> X6
- TP6 pad Y: Net-(TP6-PadY) -> Y0
- TP7 pad X: Net-(TP7-PadX) -> X4
- TP7 pad Y: Net-(TP7-PadY) -> Y0
- TP8 pad X: Net-(TP8-PadX) -> Net-(TP17-PadX)
- TP8 pad Y: Net-(TP8-PadY) -> Y3
- TP9 pad X: Net-(TP9-PadX) -> X1
- TP9 pad Y: Net-(TP9-PadY) -> Y4
- U1 pad 1: (no net) -> MOSI_5V
- U1 pad 17: Net-(C3-Pad1) -> Net-(C16-Pad1)
- U1 pad 27: Net-(C3-Pad1) -> Net-(C16-Pad1)
- U1 pad 29: Net-(C3-Pad1) -> Net-(C16-Pad1)
- U1 pad 3: (no net) -> SCK_5V
- U1 pad 38: Net-(C3-Pad1) -> Net-(C16-Pad1)
- U1 pad 4: Net-(C3-Pad1) -> Net-(C16-Pad1)
- U1 pad 40: (no net) -> Net-(D1-Pad2)
- U1 pad 5: Net-(C3-Pad1) -> Net-(C16-Pad1)
- U2 pad 10: (no net) -> SCK_3v3
- U2 pad 11: (no net) -> SCK_5V
- U2 pad 3: (no net) -> RX_3V3
- U2 pad 5: (no net) -> MOSI_5V
- U2 pad 6: MISO_5V -> MOSI_3V3
- U3 pad 10: (no net) -> MISO_5V
- U3 pad 11: (no net) -> MISO_3V3
- U3 pad 4: (no net) -> TX_3V3
- U3 pad 5: (no net) -> DRDY_3V3
Routing:
- net Net-(TP4-PadX): track 654.0 -> 0.00 mm, vias 20 -> 0
- net GND: track 647.6 -> 0.00 mm, vias 17 -> 1
- net LOAD: track 207.1 -> 0.00 mm, vias 4 -> 0
- net SERDAT_OUT_1: track 128.3 -> 0.00 mm, vias 2 -> 0
- net Net-(R22-Pad2): track 122.3 -> 0.00 mm, vias 1 -> 0
- net Net-(R15-Pad2): track 102.1 -> 0.00 mm, vias 1 -> 0
- net Net-(R25-Pad2): track 73.6 -> 0.00 mm, vias 1 -> 0
- net SERDAT_OUT_2: track 73.2 -> 0.00 mm
- net Net-(R2-Pad2): track 69.5 -> 0.00 mm, vias 1 -> 0
- net Net-(R7-Pad2): track 55.6 -> 0.00 mm, vias 1 -> 0
- net Net-(R11-Pad2): track 52.6 -> 0.00 mm, vias 3 -> 0
- net Net-(R17-Pad2): track 51.3 -> 0.00 mm, vias 1 -> 0
- net Net-(R6-Pad2): track 48.9 -> 0.00 mm, vias 1 -> 0
- net Net-(R4-Pad2): track 46.8 -> 0.00 mm, vias 1 -> 0
- net SERDAT_OUT: track 46.7 -> 0.00 mm, vias 2 -> 0
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- removed copper zone on F.Cu, net +3V3
- removed copper zone on B.Cu, net GND
Other:
- outline, holes or cut-outs redrawn
- board text removed: "3V3"
- board text removed: "CLK"
- board text removed: "GND"
- board text removed: "LOAD"
- board text removed: "SERDAT"

Commit message: Updates
Parts:
- added JP1: Jumper, Jumper:SolderJumper-2_P1.3mm_Open_TrianglePad1.0x1.5mm, B.Cu at (103.9, 139.0)
- added JP2: Jumper, Jumper:SolderJumper-2_P1.3mm_Open_TrianglePad1.0x1.5mm, B.Cu at (97.7, 138.9)
- added U4: cd40109, Package_SO:SOP-24_7.5x15.4mm_P1.27mm, B.Cu at (115.2, 130.8)
- D2, R22: moved to B.Cu
- moved C17 121.7 mm to (207.5, 137.5), turned to 180 degrees
- moved C16 118.3 mm to (205.0, 131.9), turned to 180 degrees
- moved C13 88.6 mm to (126.2, 131.2), turned to 90 degrees
- moved R22 85.0 mm to (33.1, 113.2), turned to 90 degrees
- moved D2 78.3 mm to (33.0, 108.3), turned to 90 degrees
- moved C2 61.5 mm to (206.4, 140.4)
- moved Y1 42.6 mm to (194.0, 138.7), turned to 0 degrees
- moved R1 40.4 mm to (226.0, 140.2), turned to 180 degrees
- moved C1 39.2 mm to (181.5, 140.2), turned to 180 degrees
- moved R7 34.8 mm to (193.2, 113.8), turned to 90 degrees
- moved D1 31.5 mm to (221.5, 140.2), turned to 180 degrees
- moved C5 28.7 mm to (215.3, 137.7), turned to 180 degrees
- moved C12 28.3 mm to (102.3, 130.8), turned to 90 degrees
- moved C4 24.8 mm to (196.0, 117.9), turned to 90 degrees
- moved C3 22.2 mm to (193.9, 117.9), turned to 90 degrees
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Connections:
- J1 pad 10: (no net) -> DBG_DATA_3V3
- J1 pad 12: (no net) -> WS_3V3
- J1 pad 3: RX_3V3 -> +3V3
- J1 pad 4: TX_3V3 -> RX_3V3
- J1 pad 5: DRDY_3V3 -> TX_3V3
- J1 pad 6: MOSI_3V3 -> DRDY_3V3
- J1 pad 7: SCK_3v3 -> MOSI_3V3
- J1 pad 8: MISO_3V3 -> (no net)
- J1 pad 9: (no net) -> MISO_3V3
- R11 pad 2: (no net) -> X2
- R16 pad 2: Y0 -> Y3
- R17 pad 2: Y1 -> Y2
- R18 pad 2: Y2 -> Y1
- R19 pad 2: Y3 -> Y0
- TP24 pad Y: Net-(TP24-PadY) -> Y2
- TP28 pad X: Net-(TP28-PadX) -> X4
- U1 pad 11: (no net) -> WS_5V
- U1 pad 40: Net-(D1-Pad2) -> Net-(JP1-Pad2)
- U1 pad 43: (no net) -> DBG_CLK_5V
- U2 pad 10: SCK_3v3 -> (no net)
- U2 pad 13: (no net) -> WS_5V
- U2 pad 14: (no net) -> WS_3V3
- U2 pad 15: (no net) -> +3V3
- U2 pad 2: (no net) -> +3V3
- U2 pad 7: (no net) -> +3V3
- U2 pad 9: (no net) -> +3V3
- U3 pad 13: (no net) -> DBG_DATA_3V3
- U3 pad 14: (no net) -> DBG_DATA_5V
- U3 pad 15: (no net) -> +5V
- U3 pad 2: (no net) -> +5V
- U3 pad 7: (no net) -> +5V
- U3 pad 9: (no net) -> +5V
Routing:
- net GND: track 0.00 -> 339.0 mm, vias 1 -> 23
- net Y0: track 0.00 -> 293.4 mm, vias 0 -> 6
- net +5V: track 0.00 -> 293.4 mm, vias 0 -> 19
- net X7: track 0.00 -> 270.8 mm, vias 0 -> 3
- net Net-(C16-Pad1): track 0.00 -> 249.6 mm, vias 0 -> 10
- net Y1: track 0.00 -> 200.0 mm, vias 0 -> 8
- net MOSI_5V: track 0.00 -> 161.8 mm, vias 0 -> 2
- net X6: track 0.00 -> 154.2 mm, vias 0 -> 5
- net +3V3: track 0.00 -> 153.7 mm, vias 0 -> 12
- net RX_5V: track 0.00 -> 152.5 mm, vias 0 -> 4
- net DRDY_5V: track 0.00 -> 150.6 mm, vias 0 -> 4
- net SCK_5V: track 0.00 -> 145.3 mm, vias 0 -> 2
- net Y3: track 0.00 -> 136.4 mm, vias 0 -> 3
- net Y2: track 0.00 -> 134.8 mm, vias 0 -> 5
- net X5: track 0.00 -> 131.1 mm, vias 0 -> 3
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- added copper zone on B.Cu, net GND
Other:
- outline, holes or cut-outs redrawn
- board text added: "CHECK"
- board text added: "Experimental School's Computer QT Touch Keyboard May 2024 menadue@gmail.com V1.0"
- board text removed: "Experimental School's Computer May 2024 menadue@gmail.com V1.0"

Commit message: Updates
Parts:
- C16: value C_Small -> 100uF
- C17, C3, C4, C5: value C_Small -> 100nF
- JP1: value Jumper -> DBG_LED
- JP2: value Jumper -> DBG_DATA
- U2, U3, U4: footprint Package_SO:SOP-24_7.5x15.4mm_P1.27mm -> Package_SO:SOIC-16W_7.5x10.3mm_P1.27mm
Routing:
- net X7: track 270.8 -> 386.5 mm
- net Y1: track 200.0 -> 224.2 mm
- net GND: track 339.0 -> 352.4 mm, vias 23 -> 25
- net MISO_3V3: track 108.2 -> 121.5 mm, vias 4 -> 6
- net +3V3: track 153.7 -> 166.3 mm, vias 12 -> 16
- net DBG_DATA_5V: track 3.57 -> 15.3 mm, vias 0 -> 2
- net WS_5V: track 128.9 -> 140.4 mm, vias 2 -> 4
- net +5V: track 293.4 -> 304.8 mm, vias 19 -> 21
- net Y0: track 293.4 -> 304.3 mm
- net WS_3V3: track 101.1 -> 92.8 mm
- net MISO_5V: track 120.4 -> 112.3 mm
- net DBG_DATA_3V3: track 118.0 -> 110.2 mm
- net SCK_5V: track 145.3 -> 138.9 mm, vias 2 -> 4
- net DRDY_3V3: track 90.0 -> 93.4 mm, vias 4 -> 5
- net TX_5V: track 121.7 -> 125.0 mm, vias 2 -> 4
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Other:
- board text added: "Experimental School's Computer QT Touch Keyboard May 2024 menadue@gmail.com V1.1"
- board text removed: "Experimental School's Computer QT Touch Keyboard May 2024 menadue@gmail.com V1.0"

Commit message: Updates
Parts:
- D2: value D -> ss36
- R10, R11, R12, R13, R14, R15, R16, R17, R18, R19, R20, R21, R7, R8: value R_Small -> 1k
- R2: value R_Small -> 407k
- R22: value R_Small -> 0R
- R3, R4, R5, R6, R9: value R_Small -> 470k

Commit message: Updates
Parts:
- added C18: 25uF, Capacitor_SMD:C_1206_3216Metric_Pad1.33x1.80mm_HandSolder, B.Cu at (211.4, 130.2)
- added C19: 25uF, Capacitor_SMD:C_1206_3216Metric_Pad1.33x1.80mm_HandSolder, B.Cu at (211.4, 135.2)
- added C20: 25uF, Capacitor_SMD:C_1206_3216Metric_Pad1.33x1.80mm_HandSolder, B.Cu at (211.4, 132.7)
- added C21: 25uF, Capacitor_SMD:C_1206_3216Metric_Pad1.33x1.80mm_HandSolder, B.Cu at (211.5, 127.7)
- C10, C11, C6, C7, C8, C9: value C_Small -> 4n7
- C16: footprint Capacitor_SMD:C_0805_2012Metric_Pad1.18x1.45mm_HandSolder -> Capacitor_SMD:C_1206_3216Metric_Pad1.33x1.80mm_HandSolder
- C17: value 100nF -> 25uF; footprint Capacitor_SMD:C_0805_2012Metric_Pad1.18x1.45mm_HandSolder -> Capacitor_SMD:C_1206_3216Metric_Pad1.33x1.80mm_HandSolder
- TP1: value Touchpad_qt -> A
- TP10: value Touchpad_qt -> LOAD ADDR
- TP11: value Touchpad_qt -> INCR ADDR
- TP12: value Touchpad_qt -> STOP
- TP13: value Touchpad_qt -> 7
- TP14: value Touchpad_qt -> 1
- TP15: value Touchpad_qt -> RELOAD
- TP16: value Touchpad_qt -> CLEAR
- TP17: value Touchpad_qt -> DUMP
- TP18: value Touchpad_qt -> 4
- TP19: value Touchpad_qt -> 2
- TP2: value Touchpad_qt -> LOAD IAR
- TP20: value Touchpad_qt -> CHECK
- TP21: value Touchpad_qt -> 8
- TP22: value Touchpad_qt -> MINUS
- TP23: value Touchpad_qt -> 5
- TP24: value Touchpad_qt -> 3
- TP25: value Touchpad_qt -> 9
- TP26: value Touchpad_qt -> DOT
- TP27: value Touchpad_qt -> 6
- TP28: value Touchpad_qt -> 0
- TP3: value Touchpad_qt -> DECR ADDR
- TP4: value Touchpad_qt -> B
- TP5: value Touchpad_qt -> KI RESET
- TP6: value Touchpad_qt -> LOAD STORE
- TP7: value Touchpad_qt -> NORM RESET
- TP8: value Touchpad_qt -> RUN
- TP9: value Touchpad_qt -> C
- moved R21 0.97 mm to (209.7, 124.7)
- moved C16 0.40 mm to (205.4, 131.9)
Connections:
- TP1 pad X: X3 -> X0
- TP1 pad Y: Y3 -> Y0
- TP10 pad Y: Y0 -> Y3
- TP11 pad Y: Y0 -> Y3
- TP13 pad X: X4 -> X1
- TP13 pad Y: Y1 -> Y2
- TP14 pad X: X6 -> X0
- TP14 pad Y: Y1 -> Y2
- TP16 pad X: X7 -> X3
- TP16 pad Y: Y1 -> Y2
- TP17 pad X: Net-(TP17-PadX) -> X3
- TP18 pad X: X5 -> X2
- TP18 pad Y: Y1 -> Y2
- TP19 pad Y: Y1 -> Y2
- TP2 pad X: X7 -> X0
- TP2 pad Y: Y0 -> Y3
- TP21 pad Y: Y1 -> Y2
- TP22 pad Y: Y1 -> X2
- TP23 pad Y: Y1 -> Y2
- TP24 pad Y: Y2 -> Y1
- TP25 pad Y: Y2 -> Y1
- TP26 pad Y: Y2 -> Y1
- TP27 pad Y: Y2 -> Y1
- TP28 pad X: X4 -> X0
- TP28 pad Y: Y2 -> Y1
- TP3 pad X: X5 -> X4
- TP3 pad Y: Y0 -> Y3
- TP4 pad Y: Y3 -> Y0
- TP6 pad Y: Y0 -> Y3
- TP7 pad X: X4 -> X2
- TP7 pad Y: Y0 -> Y3
- TP8 pad X: Net-(TP17-PadX) -> X3
- TP8 pad Y: Y3 -> Y0
Routing:
- net X0: track 19.1 -> 331.5 mm, vias 1 -> 9
- net X3: track 81.6 -> 300.2 mm, vias 1 -> 7
- net X2: track 61.5 -> 230.9 mm, vias 3 -> 10
- net Y0: track 304.3 -> 159.7 mm, vias 6 -> 7
- net Y3: track 136.4 -> 264.7 mm, vias 3 -> 8
- net X1: track 115.5 -> 230.3 mm, vias 1 -> 6
- net X4: track 98.5 -> 204.9 mm, vias 3 -> 4
- net X7: track 386.5 -> 304.5 mm, vias 3 -> 1
- net Net-(TP17-PadX): track 80.6 -> 0.00 mm
- net Y2: track 137.2 -> 215.8 mm, vias 5 -> 11
- net Y1: track 224.2 -> 161.0 mm, vias 8 -> 12
- net GND: track 352.4 -> 380.2 mm, vias 25 -> 28
- net X5: track 131.1 -> 123.9 mm
- net Net-(C16-Pad1): track 249.6 -> 255.8 mm
- net X6: track 154.2 -> 160.1 mm, vias 5 -> 3
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- removed copper zone on B.Cu, net GND
Other:
- board text added: "Experimental School's Computer QT Touch Keyboard June 2024 menadue@gmail.com V2.0"
- board text removed: "Experimental School's Computer QT Touch Keyboard May 2024 menadue@gmail.com V1.1"

Commit message: Updates
Connections:
- TP22 pad Y: X2 -> Y2
Routing:
- net Y2: track 215.8 -> 239.8 mm, vias 11 -> 12
- net X2: track 230.9 -> 212.0 mm, vias 10 -> 9
- net GND: track 380.2 -> 379.8 mm, vias 28 -> 29
- added copper zone on B.Cu, net GND
Other:
- board text added: "Experimental School's Computer QT Touch Keyboard July 2024 menadue@gmail.com V2.1"
- board text removed: "Experimental School's Computer QT Touch Keyboard June 2024 menadue@gmail.com V2.0"
