File: pcbs/touch_keyboard/touch_with_qt/qt_touch1/qt_touch1.sch (KiCad schematic (older format))
At the start: 36 parts, among them J1 Conn_01x12_Female, U1 QT1481, Y1 16MHz

Commit message: Updates
Parts:
- C1, C2: value C_Small -> 20pF
- Y1: footprint (none) -> Crystal:Crystal_SMD_HC49-SD_HandSoldering
Connections:
- net MOSI_5V: now reaches U1.1 (MOSI)
- net TX_5V: now reaches U1.10 (TX)
- net MISO_5V: now reaches U1.2 (MISO)
- net SCK_5V: now reaches U1.3 (SCK)
- net DRDY_5V: now reaches U1.41 (nDRDY)
- net RX_5V: now reaches U1.9 (RX)
- net Y5: now reaches R21.2
- net Y4: now reaches R20.2
- net Y3: now reaches R19.2
- net Y2: now reaches R18.2
- net Y1: now reaches R17.2
- net Y0: now reaches R16.2
- net X0: now reaches R15.2
- net X1: now reaches R13.2
- net X3: now reaches R8.2
- net X4: now reaches R14.2
- net X5: now reaches R12.2
- net X6: now reaches R10.2
- net X7: now reaches R7.2
- net RX_3V3: now reaches J1.3 (Pin_3)
- net TX_3V3: now reaches J1.4 (Pin_4)
- net DRDY_3V3: now reaches J1.5 (Pin_5)
- net MOSI_3V3: now reaches J1.6 (Pin_6)
- net SCK_3v3: now reaches J1.7 (Pin_7)
- net MISO_3V3: now reaches J1.8 (Pin_8)
Changed lines of the file:
@@
 F 0 "Y1" V 1475 4150 50  0000 L CNN
 F 1 "16MHz" V 1550 4150 50  0000 L CNN
-F 2 "" H 1775 4350 50  0001 C CNN
+F 2 "Crystal:Crystal_SMD_HC49-SD_HandSoldering" H 1775 4350 50  0001 C CNN
 F 3 "~" H 1775 4350 50  0001 C CNN
 	1    1775 4350
@@
 P 1175 4525
 F 0 "C1" H 1267 4571 50  0000 L CNN
-F 1 "C_Small" H 1267 4480 50  0000 L CNN
+F 1 "20pF" H 1267 4480 50  0000 L CNN
 F 2 "ajm_kicad:qt_touch_12_x_12" H 1175 4525 50  0001 C CNN
 F 3 "~" H 1175 4525 50  0001 C CNN
@@
 P 1775 4775
 F 0 "C2" H 1867 4821 50  0000 L CNN
-F 1 "C_Small" H 1867 4730 50  0000 L CNN
+F 1 "20pF" H 1867 4730 50  0000 L CNN
 F 2 "ajm_kicad:qt_touch_12_x_12" H 1775 4775 50  0001 C CNN
 F 3 "~" H 1775 4775 50  0001 C CNN
@@
 F1 "keys.sch" 50
 $EndSheet
+Text GLabel 3375 4000 0    50   Input ~ 0
+DRDY_5V
+Text GLabel 3375 3700 0    50   Input ~ 0
+TX_5V
+Text GLabel 3375 3600 0    50   Input ~ 0
+RX_5V
+Text GLabel 1175 1550 2    50   Input ~ 0
+RX_3V3
+Text GLabel 1175 1650 2    50   Input ~ 0
+TX_3V3
+Text GLabel 1175 1750 2    50   Input ~ 0
+DRDY_3V3
+Text GLabel 3375 3200 0    50   Input ~ 0
+MOSI_5V
+Text GLabel 3375 3300 0    50   Input ~ 0
+MISO_5V
+Text GLabel 3375 3400 0    50   Input ~ 0
+SCK_5V
+Text GLabel 1175 1850 2    50   Input ~ 0
+MOSI_3V3
+Text GLabel 1175 1950 2    50   Input ~ 0
+SCK_3v3
+Text GLabel 1175 2050 2    50   Input ~ 0
+MISO_3V3
+Text GLabel 7475 3600 2    50   Input ~ 0
+X0
+Text GLabel 7475 3500 2    50   Input ~ 0
+X1
+Text GLabel 7475 3400 2    50   Input ~ 0
+X2
+Text GLabel 7475 3300 2    50   Input ~ 0
+X3
+Text GLabel 7475 3200 2    50   Input ~ 0
+X4
+Text GLabel 7475 3100 2    50   Input ~ 0
+X5
+Text GLabel 7475 3000 2    50   Input ~ 0
+X6
+Text GLabel 7475 2900 2    50   Input ~ 0
+X7
+Wire Wire Line
+	6550 3600 7475 3600
+Wire Wire Line
+	7475 3500 6250 3500
+Wire Wire Line
+	5975 3400 7475 3400
+Wire Wire Line
+	7475 3300 5650 3300
+Wire Wire Line
+	6550 3200 7475 3200
+Wire Wire Line
+	7475 3100 6250 3100
+Wire Wire Line
+	5950 3000 7475 3000
+Wire Wire Line
+	7475 2900 5650 2900
+Text GLabel 8000 3800 2    50   Input ~ 0
+Y0
+Text GLabel 8000 4000 2    50   Input ~ 0
+Y1
+Text GLabel 8000 4200 2    50   Input ~ 0
+Y2
+Text GLabel 8000 4400 2    50   Input ~ 0
+Y3
+Text GLabel 8000 4600 2    50   Input ~ 0
+Y4
+Text GLabel 8000 4800 2    50   Input ~ 0
+Y5
+Wire Wire Line
+	8000 3800 6925 3800
+Wire Wire Line
+	6925 4000 8000 4000
+Wire Wire Line
+	8000 4200 6925 4200
+Wire Wire Line
+	8000 4400 6925 4400
+Wire Wire Line
+	8000 4600 6925 4600
+Wire Wire Line
+	6925 4800 8000 4800
 $EndSCHEMATC

Commit message: Updates
Parts:
- added C16, C17: C_Small, Capacitor_SMD:C_0805_2012Metric_Pad1.18x1.45mm_HandSolder, symbol Device:C_Small
- added D2: D, LED_SMD:LED_0805_2012Metric_Pad1.15x1.40mm_HandSolder, symbol Device:D
- added R22: R_Small, Resistor_SMD:R_0805_2012Metric_Pad1.20x1.40mm_HandSolder, symbol Device:R_Small
- C1, C10, C11, C2, C3, C4, C5, C6, C7, C8, C9: footprint ajm_kicad:qt_touch_12_x_12 -> Capacitor_SMD:C_0805_2012Metric_Pad1.18x1.45mm_HandSolder
- D1: footprint (none) -> LED_SMD:LED_0805_2012Metric_Pad1.15x1.40mm_HandSolder
- J1: footprint (none) -> Connector_PinSocket_2.54mm:PinSocket_1x12_P2.54mm_Vertical_SMD_Pin1Left
Connections:
- net +5V: now also D2.2 (A)
- net GND: now also C16.2, C17.2
- net at C3.1, C4.1, C5.1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: now also C16.1, C17.1, R22.1
- new net: D2.1 (K), R22.2
Changed lines of the file:
@@
 F 0 "C5" H 5817 2021 50  0000 L CNN
 F 1 "C_Small" H 5817 1930 50  0000 L CNN
-F 2 "ajm_kicad:qt_touch_12_x_12" H 5725 1975 50  0001 C CNN
+F 2 "Capacitor_SMD:C_0805_2012Metric_Pad1.18x1.45mm_HandSolder" H 5725 1975 50  0001 C CNN
 F 3 "~" H 5725 1975 50  0001 C CNN
 	1    5725 1975
@@
 F 0 "D1" H 2743 4317 50  0000 C CNN
 F 1 "LED" H 2743 4226 50  0000 C CNN
-F 2 "" H 2750 4100 50  0001 C CNN
+F 2 "LED_SMD:LED_0805_2012Metric_Pad1.15x1.40mm_HandSolder" H 2750 4100 50  0001 C CNN
 F 3 "~" H 2750 4100 50  0001 C CNN
 	1    2750 4100
@@
 F 0 "C3" H 4917 2021 50  0000 L CNN
 F 1 "C_Small" H 4917 1930 50  0000 L CNN
-F 2 "ajm_kicad:qt_touch_12_x_12" H 4825 1975 50  0001 C CNN
+F 2 "Capacitor_SMD:C_0805_2012Metric_Pad1.18x1.45mm_HandSolder" H 4825 1975 50  0001 C CNN
 F 3 "~" H 4825 1975 50  0001 C CNN
 	1    4825 1975
@@
 F 0 "C4" H 5342 2021 50  0000 L CNN
 F 1 "C_Small" H 5342 1930 50  0000 L CNN
-F 2 "ajm_kicad:qt_touch_12_x_12" H 5250 1975 50  0001 C CNN
+F 2 "Capacitor_SMD:C_0805_2012Metric_Pad1.18x1.45mm_HandSolder" H 5250 1975 50  0001 C CNN
 F 3 "~" H 5250 1975 50  0001 C CNN
 	1    5250 1975
@@
 F 0 "C1" H 1267 4571 50  0000 L CNN
 F 1 "20pF" H 1267 4480 50  0000 L CNN
-F 2 "ajm_kicad:qt_touch_12_x_12" H 1175 4525 50  0001 C CNN
+F 2 "Capacitor_SMD:C_0805_2012Metric_Pad1.18x1.45mm_HandSolder" H 1175 4525 50  0001 C CNN
 F 3 "~" H 1175 4525 50  0001 C CNN
 	1    1175 4525
@@
 F 0 "C2" H 1867 4821 50  0000 L CNN
 F 1 "20pF" H 1867 4730 50  0000 L CNN
-F 2 "ajm_kicad:qt_touch_12_x_12" H 1775 4775 50  0001 C CNN
+F 2 "Capacitor_SMD:C_0805_2012Metric_Pad1.18x1.45mm_HandSolder" H 1775 4775 50  0001 C CNN
 F 3 "~" H 1775 4775 50  0001 C CNN
 	1    1775 4775
@@
 F 0 "C11" V 5950 5050 50  0000 C CNN
 F 1 "C_Small" V 5950 5275 50  0000 C CNN
-F 2 "ajm_kicad:qt_touch_12_x_12" H 6000 4900 50  0001 C CNN
+F 2 "Capacitor_SMD:C_0805_2012Metric_Pad1.18x1.45mm_HandSolder" H 6000 4900 50  0001 C CNN
 F 3 "~" H 6000 4900 50  0001 C CNN
 	1    6000 4900
@@
 F 0 "C10" V 5950 4850 50  0000 C CNN
 F 1 "C_Small" V 5950 5075 50  0000 C CNN
-F 2 "ajm_kicad:qt_touch_12_x_12" H 6000 4700 50  0001 C CNN
+F 2 "Capacitor_SMD:C_0805_2012Metric_Pad1.18x1.45mm_HandSolder" H 6000 4700 50  0001 C CNN
 F 3 "~" H 6000 4700 50  0001 C CNN
 	1    6000 4700
@@
 F 0 "C9" V 5950 4650 50  0000 C CNN
 F 1 "C_Small" V 5950 4875 50  0000 C CNN
-F 2 "ajm_kicad:qt_touch_12_x_12" H 6000 4500 50  0001 C CNN
+F 2 "Capacitor_SMD:C_0805_2012Metric_Pad1.18x1.45mm_HandSolder" H 6000 4500 50  0001 C CNN
 F 3 "~" H 6000 4500 50  0001 C CNN
 	1    6000 4500
@@
 F 0 "C8" V 5950 4450 50  0000 C CNN
 F 1 "C_Small" V 5950 4675 50  0000 C CNN
-F 2 "ajm_kicad:qt_touch_12_x_12" H 6000 4300 50  0001 C CNN
+F 2 "Capacitor_SMD:C_0805_2012Metric_Pad1.18x1.45mm_HandSolder" H 6000 4300 50  0001 C CNN
 F 3 "~" H 6000 4300 50  0001 C CNN
 	1    6000 4300
@@
 F 0 "C7" V 5950 4250 50  0000 C CNN
 F 1 "C_Small" V 5950 4475 50  0000 C CNN
-F 2 "ajm_kicad:qt_touch_12_x_12" H 6000 4100 50  0001 C CNN
+F 2 "Capacitor_SMD:C_0805_2012Metric_Pad1.18x1.45mm_HandSolder" H 6000 4100 50  0001 C CNN
 F 3 "~" H 6000 4100 50  0001 C CNN
 	1    6000 4100
@@
 F 0 "C6" V 5950 4050 50  0000 C CNN
 F 1 "C_Small" V 5950 4275 50  0000 C CNN
-F 2 "ajm_kicad:qt_touch_12_x_12" H 6000 3900 50  0001 C CNN
+F 2 "Capacitor_SMD:C_0805_2012Metric_Pad1.18x1.45mm_HandSolder" H 6000 3900 50  0001 C CNN
 F 3 "~" H 6000 3900 50  0001 C CNN
 	1    6000 3900
@@
 L power:+5V #PWR0105
 U 1 1 664C8917
-P 2275 1125
-F 0 "#PWR0105" H 2275 975 50  0001 C CNN
-F 1 "+5V" H 2290 1298 50  0000 C CNN
-F 2 "" H 2275 1125 50  0001 C CNN
-F 3 "" H 2275 1125 50  0001 C CNN
-	1    2275 1125
-	1    0    0    -1
-$EndComp
-Wire Wire Line
-	3875 1300 3875 1525
+P 2275 700
+F 0 "#PWR0105" H 2275 550 50  0001 C CNN
+F 1 "+5V" H 2290 873 50  0000 C CNN
+F 2 "" H 2275 700 50  0001 C CNN
+F 3 "" H 2275 700 50  0001 C CNN
+	1    2275 700
+	1    0    0    -1
+$EndComp
 Connection ~ 3875 1525
 Wire Wire Line
@@
 $EndComp
 Wire Wire Line
-	2275 1350 2275 1125
+	2275 1350 2275 900
 Wire Wire Line
 	1175 1350 2275 1350
@@
 F 0 "J1" H 867 2535 50  0000 C CNN
 F 1 "Conn_01x12_Female" H 867 2444 50  0000 C CNN
-F 2 "" H 975 1850 50  0001 C CNN
+F 2 "Connector_PinSocket_2.54mm:PinSocket_1x12_P2.54mm_Vertical_SMD_Pin1Left" H 975 1850 50  0001 C CNN
 F 3 "~" H 975 1850 50  0001 C CNN
 	1    975  1850
@@
 Wire Wire Line
 	6925 4800 8000 4800
+$Comp
+L Device:D D2
+U 1 1 664B96E2
+P 2650 900
+F 0 "D2" H 2650 683 50  0000 C CNN
+F 1 "D" H 2650 774 50  0000 C CNN
+F 2 "LED_SMD:LED_0805_2012Metric_Pad1.15x1.40mm_HandSolder" H 2650 900 50  0001 C CNN
+F 3 "~" H 2650 900 50  0001 C CNN
+	1    2650 900
+	-1   0    0    1
+$EndComp
+Wire Wire Line
+	2500 900  2275 900
+Connection ~ 2275 900
+Wire Wire Line
+	2275 900  2275 700
+Wire Wire Line
+	3875 900  3875 1525
+$Comp
+L Device:C_Small C16
+U 1 1 664D2675
+P 4175 1075
+F 0 "C16" H 4267 1121 50  0000 L CNN
+F 1 "C_Small" H 4267 1030 50  0000 L CNN
+F 2 "Capacitor_SMD:C_0805_2012Metric_Pad1.18x1.45mm_HandSolder" H 4175 1075 50  0001 C CNN
+F 3 "~" H 4175 1075 50  0001 C CNN
+	1    4175 1075
+	1    0    0    -1
+$EndComp
+$Comp
+L Device:C_Small C17
+U 1 1 664D8C28
+P 4675 1075
+F 0 "C17" H 4767 1121 50  0000 L CNN
+F 1 "C_Small" H 4767 1030 50  0000 L CNN
+F 2 "Capacitor_SMD:C_0805_2012Metric_Pad1.18x1.45mm_HandSolder" H 4675 1075 50  0001 C CNN
+F 3 "~" H 4675 1075 50  0001 C CNN
+	1    4675 1075
+	1    0    0    -1
+$EndComp
+Wire Wire Line
+	4175 975  4175 900
+Wire Wire Line
+	4175 900  3875 900
+Wire Wire Line
+	4175 900  4675 900
+Wire Wire Line
+	4675 900  4675 975
+Connection ~ 4175 900
+$Comp
+L power:GND #PWR0108
+U 1 1 664EBBC5
+P 4675 1225
+F 0 "#PWR0108" H 4675 975 50  0001 C CNN
+F 1 "GND" H 4680 1052 50  0000 C CNN
+F 2 "" H 4675 1225 50  0001 C CNN
+F 3 "" H 4675 1225 50  0001 C CNN
+	1    4675 1225
+	1    0    0    -1
+$EndComp
+$Comp
+L power:GND #PWR0109
+U 1 1 664F1FDF
+P 4175 1225
+F 0 "#PWR0109" H 4175 975 50  0001 C CNN
+F 1 "GND" H 4180 1052 50  0000 C CNN
+F 2 "" H 4175 1225 50  0001 C CNN
+F 3 "" H 4175 1225 50  0001 C CNN
+	1    4175 1225
+	1    0    0    -1
+$EndComp
+Wire Wire Line
+	4175 1225 4175 1175
+Wire Wire Line
+	4675 1225 4675 1175
+$Comp
+L Device:R_Small R22
+U 1 1 6650BD73
+P 3275 900
+F 0 "R22" V 3079 900 50  0000 C CNN
+F 1 "R_Small" V 3170 900 50  0000 C CNN
+F 2 "Resistor_SMD:R_0805_2012Metric_Pad1.20x1.40mm_HandSolder" H 3275 900 50  0001 C CNN
+F 3 "~" H 3275 900 50  0001 C CNN
+	1    3275 900
+	0    1    1    0
+$EndComp
+Wire Wire Line
+	2800 900  3175 900
+Wire Wire Line
+	3375 900  3875 900
+Connection ~ 3875 900
 $EndSCHEMATC

Commit message: Updates
Parts:
- added JP1, JP2: Jumper, Jumper:SolderJumper-2_P1.3mm_Open_TrianglePad1.0x1.5mm, symbol Device:Jumper
Connections:
- net DRDY_3V3: now also J1.6 (Pin_6); no longer J1.5 (Pin_5)
- net MISO_3V3: now also J1.9 (Pin_9); no longer J1.8 (Pin_8)
- net MOSI_3V3: now also J1.7 (Pin_7); no longer J1.6 (Pin_6)
- net RX_3V3: now also J1.4 (Pin_4); no longer J1.3 (Pin_3)
- net SCK_3v3: now also J1.8 (Pin_8); no longer J1.7 (Pin_7)
- net TX_3V3: now also J1.5 (Pin_5); no longer J1.4 (Pin_4)
- net X2: now also R11.2
- net Y0: now also R19.2; no longer R16.2
- net Y1: now also R18.2; no longer R17.2
- net Y2: now also R17.2; no longer R18.2
- net Y3: now also R16.2; no longer R19.2
- net WS_5V: now reaches U1.11 (WS)
- net at U1.40 (nSTATUS/DBG_DATA): now also JP1.2, JP2.2; no longer D1.2 (A)
- net DBG_CLK_5V: now reaches U1.43 (S_SYNC/DBG_CLK)
- net DBG_DATA_3V3: now reaches J1.10 (Pin_10)
- net DBG_CLK_3V3: now reaches J1.11 (Pin_11)
- net WS_3V3: now reaches J1.12 (Pin_12)
- new net: D1.2 (A), JP1.1
- new net +3V3: J1.3 (Pin_3)
- new net DBG_DATA_5V: JP2.1
Other:
- moved on the sheet: D1, R1
Changed lines of the file:
@@
 L Device:LED D1
 U 1 1 664702FC
-P 2750 4100
-F 0 "D1" H 2743 4317 50  0000 C CNN
-F 1 "LED" H 2743 4226 50  0000 C CNN
-F 2 "LED_SMD:LED_0805_2012Metric_Pad1.15x1.40mm_HandSolder" H 2750 4100 50  0001 C CNN
-F 3 "~" H 2750 4100 50  0001 C CNN
-	1    2750 4100
+P 1325 3600
+F 0 "D1" H 1318 3817 50  0000 C CNN
+F 1 "LED" H 1318 3726 50  0000 C CNN
+F 2 "LED_SMD:LED_0805_2012Metric_Pad1.15x1.40mm_HandSolder" H 1325 3600 50  0001 C CNN
+F 3 "~" H 1325 3600 50  0001 C CNN
+	1    1325 3600
 	1    0    0    -1
 $EndComp
@@
 L Device:R_Small R1
 U 1 1 66471688
-P 2325 4100
-F 0 "R1" V 2521 4100 50  0000 C CNN
-F 1 "4k7" V 2430 4100 50  0000 C CNN
-F 2 "Resistor_SMD:R_0805_2012Metric_Pad1.20x1.40mm_HandSolder" H 2325 4100 50  0001 C CNN
-F 3 "~" H 2325 4100 50  0001 C CNN
-	1    2325 4100
+P 900 3600
+F 0 "R1" V 1096 3600 50  0000 C CNN
+F 1 "4k7" V 1005 3600 50  0000 C CNN
+F 2 "Resistor_SMD:R_0805_2012Metric_Pad1.20x1.40mm_HandSolder" H 900 3600 50  0001 C CNN
+F 3 "~" H 900 3600 50  0001 C CNN
+	1    900  3600
 	0    -1   -1   0
 $EndComp
@@
 L power:+5V #PWR0102
 U 1 1 664730B9
-P 1950 3950
-F 0 "#PWR0102" H 1950 3800 50  0001 C CNN
-F 1 "+5V" H 1965 4123 50  0000 C CNN
-F 2 "" H 1950 3950 50  0001 C CNN
-F 3 "" H 1950 3950 50  0001 C CNN
-	1    1950 3950
+P 700 3325
+F 0 "#PWR0102" H 700 3175 50  0001 C CNN
+F 1 "+5V" H 715 3498 50  0000 C CNN
+F 2 "" H 700 3325 50  0001 C CNN
+F 3 "" H 700 3325 50  0001 C CNN
+	1    700  3325
 	1    0    0    -1
 $EndComp
@@
 Connection ~ 3875 1525
 Wire Wire Line
-	3375 4100 2900 4100
-Wire Wire Line
-	2600 4100 2425 4100
-Wire Wire Line
-	2225 4100 1950 4100
-Wire Wire Line
-	1950 4100 1950 3950
+	1950 3600 1475 3600
+Wire Wire Line
+	1175 3600 1000 3600
 Wire Wire Line
 	3375 4300 2125 4300
@@
 L power:GND #PWR0107
 U 1 1 6651856C
-P 2400 3175
-F 0 "#PWR0107" H 2400 2925 50  0001 C CNN
-F 1 "GND" H 2405 3002 50  0000 C CNN
-F 2 "" H 2400 3175 50  0001 C CNN
-F 3 "" H 2400 3175 50  0001 C CNN
-	1    2400 3175
+P 2400 1550
+F 0 "#PWR0107" H 2400 1300 50  0001 C CNN
+F 1 "GND" H 2405 1377 50  0000 C CNN
+F 2 "" H 2400 1550 50  0001 C CNN
+F 3 "" H 2400 1550 50  0001 C CNN
+	1    2400 1550
 	1    0    0    -1
 $EndComp
@@
 $EndComp
 Wire Wire Line
-	2400 1450 2400 3175
+	2400 1450 2400 1550
 Wire Wire Line
 	1175 1450 2400 1450
@@
 Text GLabel 3375 3600 0    50   Input ~ 0
 RX_5V
-Text GLabel 1175 1550 2    50   Input ~ 0
+Text GLabel 1175 1650 2    50   Input ~ 0
 RX_3V3
-Text GLabel 1175 1650 2    50   Input ~ 0
+Text GLabel 1175 1750 2    50   Input ~ 0
 TX_3V3
-Text GLabel 1175 1750 2    50   Input ~ 0
+Text GLabel 1175 1850 2    50   Input ~ 0
 DRDY_3V3
 Text GLabel 3375 3200 0    50   Input ~ 0
@@
 Text GLabel 3375 3400 0    50   Input ~ 0
 SCK_5V
-Text GLabel 1175 1850 2    50   Input ~ 0
+Text GLabel 1175 1950 2    50   Input ~ 0
 MOSI_3V3
-Text GLabel 1175 1950 2    50   Input ~ 0
+Text GLabel 1175 2050 2    50   Input ~ 0
 SCK_3v3
-Text GLabel 1175 2050 2    50   Input ~ 0
+Text GLabel 1175 2150 2    50   Input ~ 0
 MISO_3V3
 Text GLabel 7475 3600 2    50   Input ~ 0
@@
 	7475 3500 6250 3500
 Wire Wire Line
-	5975 3400 7475 3400
-Wire Wire Line
 	7475 3300 5650 3300
 Wire Wire Line
@@
 Wire Wire Line
 	7475 2900 5650 2900
+Text GLabel 8000 4400 2    50   Input ~ 0
+Y0
+Text GLabel 8000 4200 2    50   Input ~ 0
+Y1
+Text GLabel 8000 4000 2    50   Input ~ 0
+Y2
 Text GLabel 8000 3800 2    50   Input ~ 0
-Y0
-Text GLabel 8000 4000 2    50   Input ~ 0
-Y1
-Text GLabel 8000 4200 2    50   Input ~ 0
-Y2
-Text GLabel 8000 4400 2    50   Input ~ 0
 Y3
 Text GLabel 8000 4600 2    50   Input ~ 0
@@
 	3375 900  3875 900
 Connection ~ 3875 900
+$Comp
+L Device:Jumper JP1
+U 1 1 665BE849
+P 2250 3600
+F 0 "JP1" H 1750 3775 50  0000 C CNN
+F 1 "Jumper" H 1825 3700 50  0000 C CNN
+F 2 "Jumper:SolderJumper-2_P1.3mm_Open_TrianglePad1.0x1.5mm" H 2250 3600 50  0001 C CNN
+F 3 "~" H 2250 3600 50  0001 C CNN
+	1    2250 3600
+	1    0    0    -1
+$EndComp
+$Comp
+L Device:Jumper JP2
+U 1 1 665C04AA
+P 2250 3875
+F 0 "JP2" H 1750 4050 50  0000 C CNN
+F 1 "Jumper" H 1825 3975 50  0000 C CNN
+F 2 "Jumper:SolderJumper-2_P1.3mm_Open_TrianglePad1.0x1.5mm" H 2250 3875 50  0001 C CNN
+F 3 "~" H 2250 3875 50  0001 C CNN
+	1    2250 3875
+	1    0    0    -1
+$EndComp
+Wire Wire Line
+	3375 4100 2550 4100
+Wire Wire Line
+	2550 4100 2550 3875
+Wire Wire Line
+	2550 3875 2550 3600
+Connection ~ 2550 3875
+Text GLabel 1950 3875 0    50   Input ~ 0
+DBG_DATA_5V
+Text GLabel 3375 3000 0    50   Input ~ 0
+DBG_CLK_5V
+Text GLabel 1175 2250 2    50   Input ~ 0
+DBG_DATA_3V3
+Text GLabel 1175 2350 2    50   Input ~ 0
+DBG_CLK_3V3
+Text GLabel 3375 3800 0    50   Input ~ 0
+WS_5V
+Text GLabel 1175 2450 2    50   Input ~ 0
+WS_3V3
+Wire Wire Line
+	700  3325 700  3600
+Wire Wire Line
+	700  3600 800  3600
+$Comp
+L power:+3V3 #PWR0113
+U 1 1 6660825A
+P 2075 1725
+F 0 "#PWR0113" H 2075 1575 50  0001 C CNN
+F 1 "+3V3" H 2090 1898 50  0000 C CNN
+F 2 "" H 2075 1725 50  0001 C CNN
+F 3 "" H 2075 1725 50  0001 C CNN
+	1    2075 1725
+	1    0    0    -1
+$EndComp
+Wire Wire Line
+	2075 1725 1750 1725
+Wire Wire Line
+	1750 1725 1750 1550
+Wire Wire Line
+	1750 1550 1175 1550
+Wire Wire Line
+	5950 3400 7475 3400
 $EndSCHEMATC

Commit message: Updates
Parts:
- C16: value C_Small -> 100uF
- C17, C3, C4, C5: value C_Small -> 100nF
- JP1: value Jumper -> DBG_LED
- JP2: value Jumper -> DBG_DATA
Changed lines of the file:
@@
 P 5725 1975
 F 0 "C5" H 5817 2021 50  0000 L CNN
-F 1 "C_Small" H 5817 1930 50  0000 L CNN
+F 1 "100nF" H 5817 1930 50  0000 L CNN
 F 2 "Capacitor_SMD:C_0805_2012Metric_Pad1.18x1.45mm_HandSolder" H 5725 1975 50  0001 C CNN
 F 3 "~" H 5725 1975 50  0001 C CNN
@@
 P 4825 1975
 F 0 "C3" H 4917 2021 50  0000 L CNN
-F 1 "C_Small" H 4917 1930 50  0000 L CNN
+F 1 "100nF" H 4917 1930 50  0000 L CNN
 F 2 "Capacitor_SMD:C_0805_2012Metric_Pad1.18x1.45mm_HandSolder" H 4825 1975 50  0001 C CNN
 F 3 "~" H 4825 1975 50  0001 C CNN
@@
 P 5250 1975
 F 0 "C4" H 5342 2021 50  0000 L CNN
-F 1 "C_Small" H 5342 1930 50  0000 L CNN
+F 1 "100nF" H 5342 1930 50  0000 L CNN
 F 2 "Capacitor_SMD:C_0805_2012Metric_Pad1.18x1.45mm_HandSolder" H 5250 1975 50  0001 C CNN
 F 3 "~" H 5250 1975 50  0001 C CNN
@@
 P 4175 1075
 F 0 "C16" H 4267 1121 50  0000 L CNN
-F 1 "C_Small" H 4267 1030 50  0000 L CNN
+F 1 "100uF" H 4267 1030 50  0000 L CNN
 F 2 "Capacitor_SMD:C_0805_2012Metric_Pad1.18x1.45mm_HandSolder" H 4175 1075 50  0001 C CNN
 F 3 "~" H 4175 1075 50  0001 C CNN
@@
 P 4675 1075
 F 0 "C17" H 4767 1121 50  0000 L CNN
-F 1 "C_Small" H 4767 1030 50  0000 L CNN
+F 1 "100nF" H 4767 1030 50  0000 L CNN
 F 2 "Capacitor_SMD:C_0805_2012Metric_Pad1.18x1.45mm_HandSolder" H 4675 1075 50  0001 C CNN
 F 3 "~" H 4675 1075 50  0001 C CNN
@@
 P 2250 3600
 F 0 "JP1" H 1750 3775 50  0000 C CNN
-F 1 "Jumper" H 1825 3700 50  0000 C CNN
+F 1 "DBG_LED" H 1825 3700 50  0000 C CNN
 F 2 "Jumper:SolderJumper-2_P1.3mm_Open_TrianglePad1.0x1.5mm" H 2250 3600 50  0001 C CNN
 F 3 "~" H 2250 3600 50  0001 C CNN
@@
 P 2250 3875
 F 0 "JP2" H 1750 4050 50  0000 C CNN
-F 1 "Jumper" H 1825 3975 50  0000 C CNN
+F 1 "DBG_DATA" H 1825 3975 50  0000 C CNN
 F 2 "Jumper:SolderJumper-2_P1.3mm_Open_TrianglePad1.0x1.5mm" H 2250 3875 50  0001 C CNN
 F 3 "~" H 2250 3875 50  0001 C CNN
