File: pcbs/touch_keyboard/touch_with_qt/qt_touch1/qt_touch1.sch (KiCad schematic (older format))
At the start: 42 parts, among them J1 Conn_01x12_Female, U1 QT1481, Y1 16MHz

Commit message: Updates
Parts:
- D2: value D -> ss36
- R10, R11, R12, R13, R14, R15, R16, R17, R18, R19, R20, R21, R7, R8: value R_Small -> 1k
- R2: value R_Small -> 407k
- R22: value R_Small -> 0R
- R3, R4, R5, R6, R9: value R_Small -> 470k
Changed lines of the file:
@@
 P 4925 5450
 F 0 "R2" V 4925 4725 50  0000 L CNN
-F 1 "R_Small" V 4925 4875 50  0000 L CNN
+F 1 "407k" V 4925 4875 50  0000 L CNN
 F 2 "Resistor_SMD:R_0805_2012Metric_Pad1.20x1.40mm_HandSolder" H 4925 5450 50  0001 C CNN
 F 3 "~" H 4925 5450 50  0001 C CNN
@@
 P 6825 4800
 F 0 "R21" V 6875 4525 50  0000 L CNN
-F 1 "R_Small" V 6875 4200 50  0000 L CNN
+F 1 "1k" V 6875 4200 50  0000 L CNN
 F 2 "Resistor_SMD:R_0805_2012Metric_Pad1.20x1.40mm_HandSolder" H 6825 4800 50  0001 C CNN
 F 3 "~" H 6825 4800 50  0001 C CNN
@@
 P 5075 5450
 F 0 "R3" V 5075 4725 50  0000 L CNN
-F 1 "R_Small" V 5075 4875 50  0000 L CNN
+F 1 "470k" V 5075 4875 50  0000 L CNN
 F 2 "Resistor_SMD:R_0805_2012Metric_Pad1.20x1.40mm_HandSolder" H 5075 5450 50  0001 C CNN
 F 3 "~" H 5075 5450 50  0001 C CNN
@@
 P 5225 5450
 F 0 "R4" V 5225 4725 50  0000 L CNN
-F 1 "R_Small" V 5225 4875 50  0000 L CNN
+F 1 "470k" V 5225 4875 50  0000 L CNN
 F 2 "Resistor_SMD:R_0805_2012Metric_Pad1.20x1.40mm_HandSolder" H 5225 5450 50  0001 C CNN
 F 3 "~" H 5225 5450 50  0001 C CNN
@@
 P 5375 5450
 F 0 "R5" V 5375 4725 50  0000 L CNN
-F 1 "R_Small" V 5375 4875 50  0000 L CNN
+F 1 "470k" V 5375 4875 50  0000 L CNN
 F 2 "Resistor_SMD:R_0805_2012Metric_Pad1.20x1.40mm_HandSolder" H 5375 5450 50  0001 C CNN
 F 3 "~" H 5375 5450 50  0001 C CNN
@@
 P 5525 5450
 F 0 "R6" V 5525 4725 50  0000 L CNN
-F 1 "R_Small" V 5525 4875 50  0000 L CNN
+F 1 "470k" V 5525 4875 50  0000 L CNN
 F 2 "Resistor_SMD:R_0805_2012Metric_Pad1.20x1.40mm_HandSolder" H 5525 5450 50  0001 C CNN
 F 3 "~" H 5525 5450 50  0001 C CNN
@@
 P 5675 5450
 F 0 "R9" V 5675 4725 50  0000 L CNN
-F 1 "R_Small" V 5675 4875 50  0000 L CNN
+F 1 "470k" V 5675 4875 50  0000 L CNN
 F 2 "Resistor_SMD:R_0805_2012Metric_Pad1.20x1.40mm_HandSolder" H 5675 5450 50  0001 C CNN
 F 3 "~" H 5675 5450 50  0001 C CNN
@@
 P 6825 4600
 F 0 "R20" V 6875 4325 50  0000 L CNN
-F 1 "R_Small" V 6875 4000 50  0000 L CNN
+F 1 "1k" V 6875 4000 50  0000 L CNN
 F 2 "Resistor_SMD:R_0805_2012Metric_Pad1.20x1.40mm_HandSolder" H 6825 4600 50  0001 C CNN
 F 3 "~" H 6825 4600 50  0001 C CNN
@@
 P 6825 4400
 F 0 "R19" V 6875 4125 50  0000 L CNN
-F 1 "R_Small" V 6875 3800 50  0000 L CNN
+F 1 "1k" V 6875 3800 50  0000 L CNN
 F 2 "Resistor_SMD:R_0805_2012Metric_Pad1.20x1.40mm_HandSolder" H 6825 4400 50  0001 C CNN
 F 3 "~" H 6825 4400 50  0001 C CNN
@@
 P 6825 4200
 F 0 "R18" V 6875 3925 50  0000 L CNN
-F 1 "R_Small" V 6875 3600 50  0000 L CNN
+F 1 "1k" V 6875 3600 50  0000 L CNN
 F 2 "Resistor_SMD:R_0805_2012Metric_Pad1.20x1.40mm_HandSolder" H 6825 4200 50  0001 C CNN
 F 3 "~" H 6825 4200 50  0001 C CNN
@@
 P 6825 4000
 F 0 "R17" V 6875 3725 50  0000 L CNN
-F 1 "R_Small" V 6875 3400 50  0000 L CNN
+F 1 "1k" V 6875 3400 50  0000 L CNN
 F 2 "Resistor_SMD:R_0805_2012Metric_Pad1.20x1.40mm_HandSolder" H 6825 4000 50  0001 C CNN
 F 3 "~" H 6825 4000 50  0001 C CNN
@@
 P 6825 3800
 F 0 "R16" V 6875 3525 50  0000 L CNN
-F 1 "R_Small" V 6875 3200 50  0000 L CNN
+F 1 "1k" V 6875 3200 50  0000 L CNN
 F 2 "Resistor_SMD:R_0805_2012Metric_Pad1.20x1.40mm_HandSolder" H 6825 3800 50  0001 C CNN
 F 3 "~" H 6825 3800 50  0001 C CNN
@@
 P 6450 3600
 F 0 "R15" V 6500 3325 50  0000 L CNN
-F 1 "R_Small" V 6500 3000 50  0000 L CNN
+F 1 "1k" V 6500 3000 50  0000 L CNN
 F 2 "Resistor_SMD:R_0805_2012Metric_Pad1.20x1.40mm_HandSolder" H 6450 3600 50  0001 C CNN
 F 3 "~" H 6450 3600 50  0001 C CNN
@@
 P 6150 3500
 F 0 "R13" V 6200 3225 50  0000 L CNN
-F 1 "R_Small" V 6200 2900 50  0000 L CNN
+F 1 "1k" V 6200 2900 50  0000 L CNN
 F 2 "Resistor_SMD:R_0805_2012Metric_Pad1.20x1.40mm_HandSolder" H 6150 3500 50  0001 C CNN
 F 3 "~" H 6150 3500 50  0001 C CNN
@@
 P 5850 3400
 F 0 "R11" V 5900 3125 50  0000 L CNN
-F 1 "R_Small" V 5900 2800 50  0000 L CNN
+F 1 "1k" V 5900 2800 50  0000 L CNN
 F 2 "Resistor_SMD:R_0805_2012Metric_Pad1.20x1.40mm_HandSolder" H 5850 3400 50  0001 C CNN
 F 3 "~" H 5850 3400 50  0001 C CNN
@@
 P 5550 3300
 F 0 "R8" V 5600 3025 50  0000 L CNN
-F 1 "R_Small" V 5600 2700 50  0000 L CNN
+F 1 "1k" V 5600 2700 50  0000 L CNN
 F 2 "Resistor_SMD:R_0805_2012Metric_Pad1.20x1.40mm_HandSolder" H 5550 3300 50  0001 C CNN
 F 3 "~" H 5550 3300 50  0001 C CNN
@@
 P 6450 3200
 F 0 "R14" V 6500 2925 50  0000 L CNN
-F 1 "R_Small" V 6500 2600 50  0000 L CNN
+F 1 "1k" V 6500 2600 50  0000 L CNN
 F 2 "Resistor_SMD:R_0805_2012Metric_Pad1.20x1.40mm_HandSolder" H 6450 3200 50  0001 C CNN
 F 3 "~" H 6450 3200 50  0001 C CNN
@@
 P 6150 3100
 F 0 "R12" V 6200 2825 50  0000 L CNN
-F 1 "R_Small" V 6200 2500 50  0000 L CNN
+F 1 "1k" V 6200 2500 50  0000 L CNN
 F 2 "Resistor_SMD:R_0805_2012Metric_Pad1.20x1.40mm_HandSolder" H 6150 3100 50  0001 C CNN
 F 3 "~" H 6150 3100 50  0001 C CNN
@@
 P 5850 3000
 F 0 "R10" V 5900 2725 50  0000 L CNN
-F 1 "R_Small" V 5900 2400 50  0000 L CNN
+F 1 "1k" V 5900 2400 50  0000 L CNN
 F 2 "Resistor_SMD:R_0805_2012Metric_Pad1.20x1.40mm_HandSolder" H 5850 3000 50  0001 C CNN
 F 3 "~" H 5850 3000 50  0001 C CNN
@@
 P 5550 2900
 F 0 "R7" V 5600 2625 50  0000 L CNN
-F 1 "R_Small" V 5600 2300 50  0000 L CNN
+F 1 "1k" V 5600 2300 50  0000 L CNN
 F 2 "Resistor_SMD:R_0805_2012Metric_Pad1.20x1.40mm_HandSolder" H 5550 2900 50  0001 C CNN
 F 3 "~" H 5550 2900 50  0001 C CNN
@@
 P 2650 900
 F 0 "D2" H 2650 683 50  0000 C CNN
-F 1 "D" H 2650 774 50  0000 C CNN
+F 1 "ss36" H 2650 774 50  0000 C CNN
 F 2 "LED_SMD:LED_0805_2012Metric_Pad1.15x1.40mm_HandSolder" H 2650 900 50  0001 C CNN
 F 3 "~" H 2650 900 50  0001 C CNN
@@
 P 3275 900
 F 0 "R22" V 3079 900 50  0000 C CNN
-F 1 "R_Small" V 3170 900 50  0000 C CNN
+F 1 "0R" V 3170 900 50  0000 C CNN
 F 2 "Resistor_SMD:R_0805_2012Metric_Pad1.20x1.40mm_HandSolder" H 3275 900 50  0001 C CNN
 F 3 "~" H 3275 900 50  0001 C CNN

Commit message: Updates
Parts:
- added C18, C19, C20, C21: 25uF, Capacitor_SMD:C_1206_3216Metric_Pad1.33x1.80mm_HandSolder, symbol Device:C_Small
- C10, C11, C6, C7, C8, C9: value C_Small -> 4n7
- C16: footprint Capacitor_SMD:C_0805_2012Metric_Pad1.18x1.45mm_HandSolder -> Capacitor_SMD:C_1206_3216Metric_Pad1.33x1.80mm_HandSolder
- C17: value 100nF -> 25uF; footprint Capacitor_SMD:C_0805_2012Metric_Pad1.18x1.45mm_HandSolder -> Capacitor_SMD:C_1206_3216Metric_Pad1.33x1.80mm_HandSolder
Connections:
- net GND: now also C18.2, C19.2, C20.2, C21.2
- net at C16.1, C17.1, C3.1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: now also C18.1, C19.1, C20.1, C21.1
Changed lines of the file:
@@
 P 6000 4900
 F 0 "C11" V 5950 5050 50  0000 C CNN
-F 1 "C_Small" V 5950 5275 50  0000 C CNN
+F 1 "4n7" V 5950 5275 50  0000 C CNN
 F 2 "Capacitor_SMD:C_0805_2012Metric_Pad1.18x1.45mm_HandSolder" H 6000 4900 50  0001 C CNN
 F 3 "~" H 6000 4900 50  0001 C CNN
@@
 P 6000 4700
 F 0 "C10" V 5950 4850 50  0000 C CNN
-F 1 "C_Small" V 5950 5075 50  0000 C CNN
+F 1 "4n7" V 5950 5075 50  0000 C CNN
 F 2 "Capacitor_SMD:C_0805_2012Metric_Pad1.18x1.45mm_HandSolder" H 6000 4700 50  0001 C CNN
 F 3 "~" H 6000 4700 50  0001 C CNN
@@
 P 6000 4500
 F 0 "C9" V 5950 4650 50  0000 C CNN
-F 1 "C_Small" V 5950 4875 50  0000 C CNN
+F 1 "4n7" V 5950 4875 50  0000 C CNN
 F 2 "Capacitor_SMD:C_0805_2012Metric_Pad1.18x1.45mm_HandSolder" H 6000 4500 50  0001 C CNN
 F 3 "~" H 6000 4500 50  0001 C CNN
@@
 P 6000 4300
 F 0 "C8" V 5950 4450 50  0000 C CNN
-F 1 "C_Small" V 5950 4675 50  0000 C CNN
+F 1 "4n7" V 5950 4675 50  0000 C CNN
 F 2 "Capacitor_SMD:C_0805_2012Metric_Pad1.18x1.45mm_HandSolder" H 6000 4300 50  0001 C CNN
 F 3 "~" H 6000 4300 50  0001 C CNN
@@
 P 6000 4100
 F 0 "C7" V 5950 4250 50  0000 C CNN
-F 1 "C_Small" V 5950 4475 50  0000 C CNN
+F 1 "4n7" V 5950 4475 50  0000 C CNN
 F 2 "Capacitor_SMD:C_0805_2012Metric_Pad1.18x1.45mm_HandSolder" H 6000 4100 50  0001 C CNN
 F 3 "~" H 6000 4100 50  0001 C CNN
@@
 P 6000 3900
 F 0 "C6" V 5950 4050 50  0000 C CNN
-F 1 "C_Small" V 5950 4275 50  0000 C CNN
+F 1 "4n7" V 5950 4275 50  0000 C CNN
 F 2 "Capacitor_SMD:C_0805_2012Metric_Pad1.18x1.45mm_HandSolder" H 6000 3900 50  0001 C CNN
 F 3 "~" H 6000 3900 50  0001 C CNN
@@
 F 0 "C16" H 4267 1121 50  0000 L CNN
 F 1 "100uF" H 4267 1030 50  0000 L CNN
-F 2 "Capacitor_SMD:C_0805_2012Metric_Pad1.18x1.45mm_HandSolder" H 4175 1075 50  0001 C CNN
+F 2 "Capacitor_SMD:C_1206_3216Metric_Pad1.33x1.80mm_HandSolder" H 4175 1075 50  0001 C CNN
 F 3 "~" H 4175 1075 50  0001 C CNN
 	1    4175 1075
@@
 P 4675 1075
 F 0 "C17" H 4767 1121 50  0000 L CNN
-F 1 "100nF" H 4767 1030 50  0000 L CNN
-F 2 "Capacitor_SMD:C_0805_2012Metric_Pad1.18x1.45mm_HandSolder" H 4675 1075 50  0001 C CNN
+F 1 "25uF" H 4767 1030 50  0000 L CNN
+F 2 "Capacitor_SMD:C_1206_3216Metric_Pad1.33x1.80mm_HandSolder" H 4675 1075 50  0001 C CNN
 F 3 "~" H 4675 1075 50  0001 C CNN
 	1    4675 1075
@@
 L power:GND #PWR0108
 U 1 1 664EBBC5
-P 4675 1225
-F 0 "#PWR0108" H 4675 975 50  0001 C CNN
-F 1 "GND" H 4680 1052 50  0000 C CNN
-F 2 "" H 4675 1225 50  0001 C CNN
-F 3 "" H 4675 1225 50  0001 C CNN
-	1    4675 1225
+P 4675 1275
+F 0 "#PWR0108" H 4675 1025 50  0001 C CNN
+F 1 "GND" H 4680 1102 50  0000 C CNN
+F 2 "" H 4675 1275 50  0001 C CNN
+F 3 "" H 4675 1275 50  0001 C CNN
+	1    4675 1275
 	1    0    0    -1
 $EndComp
@@
 Wire Wire Line
 	4175 1225 4175 1175
-Wire Wire Line
-	4675 1225 4675 1175
 $Comp
 L Device:R_Small R22
@@
 Wire Wire Line
 	5950 3400 7475 3400
+Connection ~ 4675 900
+Wire Wire Line
+	5225 900  5675 900
+Connection ~ 5225 900
+Connection ~ 5675 900
+Wire Wire Line
+	4675 900  5225 900
+Wire Wire Line
+	5675 900  6150 900
+Connection ~ 6150 900
+Wire Wire Line
+	6150 900  6650 900
+$Comp
+L Device:C_Small C18
+U 1 1 668C5002
+P 5225 1100
+F 0 "C18" H 5317 1146 50  0000 L CNN
+F 1 "25uF" H 5317 1055 50  0000 L CNN
+F 2 "Capacitor_SMD:C_1206_3216Metric_Pad1.33x1.80mm_HandSolder" H 5225 1100 50  0001 C CNN
+F 3 "~" H 5225 1100 50  0001 C CNN
+	1    5225 1100
+	1    0    0    -1
+$EndComp
+Wire Wire Line
+	5225 900  5225 1000
+$Comp
+L Device:C_Small C19
+U 1 1 668CCF0D
+P 5675 1100
+F 0 "C19" H 5767 1146 50  0000 L CNN
+F 1 "25uF" H 5767 1055 50  0000 L CNN
+F 2 "Capacitor_SMD:C_1206_3216Metric_Pad1.33x1.80mm_HandSolder" H 5675 1100 50  0001 C CNN
+F 3 "~" H 5675 1100 50  0001 C CNN
+	1    5675 1100
+	1    0    0    -1
+$EndComp
+Wire Wire Line
+	5675 900  5675 1000
+$Comp
+L Device:C_Small C20
+U 1 1 668D4DC5
+P 6150 1100
+F 0 "C20" H 6242 1146 50  0000 L CNN
+F 1 "25uF" H 6242 1055 50  0000 L CNN
+F 2 "Capacitor_SMD:C_1206_3216Metric_Pad1.33x1.80mm_HandSolder" H 6150 1100 50  0001 C CNN
+F 3 "~" H 6150 1100 50  0001 C CNN
+	1    6150 1100
+	1    0    0    -1
+$EndComp
+Wire Wire Line
+	6150 900  6150 1000
+$Comp
+L Device:C_Small C21
+U 1 1 668DCDD6
+P 6650 1100
+F 0 "C21" H 6742 1146 50  0000 L CNN
+F 1 "25uF" H 6742 1055 50  0000 L CNN
+F 2 "Capacitor_SMD:C_1206_3216Metric_Pad1.33x1.80mm_HandSolder" H 6650 1100 50  0001 C CNN
+F 3 "~" H 6650 1100 50  0001 C CNN
+	1    6650 1100
+	1    0    0    -1
+$EndComp
+Wire Wire Line
+	6650 900  6650 1000
+Wire Wire Line
+	5225 1200 5675 1200
+Connection ~ 5675 1200
+Wire Wire Line
+	5675 1200 6150 1200
+Connection ~ 6150 1200
+Wire Wire Line
+	6150 1200 6650 1200
+Wire Wire Line
+	4675 1175 4675 1200
+Wire Wire Line
+	5225 1200 4675 1200
+Connection ~ 5225 1200
+Connection ~ 4675 1200
+Wire Wire Line
+	4675 1200 4675 1275
 $EndSCHEMATC

Commit message: Updates
Parts:
- R2: value 407k -> 470k
Changed lines of the file:
@@
 P 4925 5450
 F 0 "R2" V 4925 4725 50  0000 L CNN
-F 1 "407k" V 4925 4875 50  0000 L CNN
+F 1 "470k" V 4925 4875 50  0000 L CNN
 F 2 "Resistor_SMD:R_0805_2012Metric_Pad1.20x1.40mm_HandSolder" H 4925 5450 50  0001 C CNN
 F 3 "~" H 4925 5450 50  0001 C CNN
